File: hw/processor.kicad_sch (KiCad schematic)
At the start: 2 parts, among them U1 ISP2454-LP-JT

Commit message: Sheet pins
Changed lines of the file:
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@@
 	(generator_version "9.0")
 	(paper "A3")
-	(hierarchical_label "SCL"
+	(hierarchical_label "PMICSCL"
 		(shape output)
 		(at 130.81 196.85 180)
@@
 		)
 	)
-	(hierarchical_label "rCOL4"
-		(shape output)
-		(at 300.99 226.06 90)
-		(effects
-			(font
-				(size 1.27 1.27)
-			)
-			(justify left)
-		)
-	)
-	(hierarchical_label "ROW1"
-		(shape input)
-		(at 60.96 252.73 90)
-		(effects
-			(font
-				(size 1.27 1.27)
-			)
-			(justify left)
-		)
-	)
-	(hierarchical_label "ROW0"
-		(shape input)
-		(at 45.72 252.73 90)
-		(effects
-			(font
-				(size 1.27 1.27)
-			)
-			(justify left)
-		)
-	)
-	(hierarchical_label "rROW0"
-		(shape input)
-		(at 297.18 241.3 90)
-		(effects
-			(font
-				(size 1.27 1.27)
-			)
-			(justify left)
-		)
-	)
-	(hierarchical_label "rROW2"
-		(shape input)
-		(at 266.7 241.3 90)
-		(effects
-			(font
-				(size 1.27 1.27)
-			)
-			(justify left)
-		)
-	)
-	(hierarchical_label "COL2"
-		(shape output)
-		(at 96.52 238.76 90)
-		(effects
-			(font
-				(size 1.27 1.27)
-			)
-			(justify left)
-		)
-	)
-	(hierarchical_label "COL5"
-		(shape output)
-		(at 58.42 238.76 90)
-		(effects
-			(font
-				(size 1.27 1.27)
-			)
-			(justify left)
-		)
-	)
-	(hierarchical_label "COL6"
-		(shape output)
-		(at 45.72 238.76 90)
-		(effects
-			(font
-				(size 1.27 1.27)
-			)
-			(justify left)
-		)
-	)
-	(hierarchical_label "COL1"
-		(shape output)
-		(at 109.22 238.76 90)
-		(effects
-			(font
-				(size 1.27 1.27)
-			)
-			(justify left)
-		)
-	)
-	(hierarchical_label "rSCL"
+	(hierarchical_label "rPMICSCL"
 		(shape output)
 		(at 255.27 157.48 180)
@@
 			)
 			(justify right)
-		)
-	)
-	(hierarchical_label "COL3"
-		(shape output)
-		(at 83.82 238.76 90)
-		(effects
-			(font
-				(size 1.27 1.27)
-			)
-			(justify left)
 		)
 	)
@@
 		)
 	)
-	(hierarchical_label "rROW3"
-		(shape input)
-		(at 251.46 241.3 90)
-		(effects
-			(font
-				(size 1.27 1.27)
-			)
-			(justify left)
-		)
-	)
-	(hierarchical_label "rCOL6"
-		(shape output)
-		(at 326.39 226.06 90)
-		(effects
-			(font
-				(size 1.27 1.27)
-			)
-			(justify left)
-		)
-	)
 	(hierarchical_label "PMICINT"
 		(shape input)
@@
 		)
 	)
-	(hierarchical_label "rCOL0"
-		(shape output)
-		(at 250.19 226.06 90)
-		(effects
-			(font
-				(size 1.27 1.27)
-			)
-			(justify left)
-		)
-	)
-	(hierarchical_label "rCOL5"
-		(shape output)
-		(at 313.69 226.06 90)
-		(effects
-			(font
-				(size 1.27 1.27)
-			)
-			(justify left)
-		)
-	)
-	(hierarchical_label "ROW2"
-		(shape input)
-		(at 76.2 252.73 90)
-		(effects
-			(font
-				(size 1.27 1.27)
-			)
-			(justify left)
-		)
-	)
-	(hierarchical_label "ROW3"
-		(shape input)
-		(at 91.44 252.73 90)
-		(effects
-			(font
-				(size 1.27 1.27)
-			)
-			(justify left)
-		)
-	)
-	(hierarchical_label "rCOL1"
-		(shape output)
-		(at 262.89 226.06 90)
-		(effects
-			(font
-				(size 1.27 1.27)
-			)
-			(justify left)
-		)
-	)
-	(hierarchical_label "rCOL2"
-		(shape output)
-		(at 275.59 226.06 90)
-		(effects
-			(font
-				(size 1.27 1.27)
-			)
-			(justify left)
-		)
-	)
-	(hierarchical_label "COL4"
-		(shape output)
-		(at 71.12 238.76 90)
-		(effects
-			(font
-				(size 1.27 1.27)
-			)
-			(justify left)
-		)
-	)
-	(hierarchical_label "rSDA"
+	(hierarchical_label "rPMICSDA"
 		(shape bidirectional)
 		(at 255.27 154.94 180)
@@
 		)
 	)
-	(hierarchical_label "SDA"
+	(hierarchical_label "PMICSDA"
 		(shape bidirectional)
 		(at 130.81 194.31 180)
@@
 		)
 	)
-	(hierarchical_label "rCOL3"
-		(shape output)
-		(at 288.29 226.06 90)
-		(effects
-			(font
-				(size 1.27 1.27)
-			)
-			(justify left)
-		)
-	)
-	(hierarchical_label "COL0"
-		(shape output)
-		(at 121.92 238.76 90)
-		(effects
-			(font
-				(size 1.27 1.27)
-			)
-			(justify left)
-		)
-	)
-	(hierarchical_label "rROW1"
-		(shape input)
-		(at 281.94 241.3 90)
-		(effects
-			(font
-				(size 1.27 1.27)
-			)
-			(justify left)
-		)
-	)
