File: hw/pmic.kicad_sch (KiCad schematic)
At the start: 40 parts, among them J1 TYPE-C-31-M-13C, J2 Conn_01x02, U2 NPM1300-QEAA-R

Commit message: all true erc errors solved
Other:
- moved on the sheet: R4, U2D
