File: hw/pmic.kicad_sch (KiCad schematic)
At the start: 38 parts, among them J1 TYPE-C-31-M-13C, J2 JST_S2B-PH-SM4-TB, U1 NPM1300-QEAA-R

Commit message: i2c eeprom
Parts:
- removed R5, R6, rR5, rR6: 10k, Alidade:R_0603_1608Metric, symbol Alidade:R
Connections:
- net PMICINT: now also U1.7 (GPIO0); no longer U1.8 (GPIO1)
- net rPMICINT: now also rU1.7 (GPIO0); no longer rU1.8 (GPIO1)
- net PMICGPIO2: no longer names the net of U1.9 (GPIO2)
- net PMICGPIO3: no longer names the net of U1.10 (GPIO3)
- net rPMICGPIO2: no longer names the net of rU1.9 (GPIO2)
- net rPMICGPIO3: no longer names the net of rU1.10 (GPIO3)
- new net PMICGPIO1: U1.8 (GPIO1)
- new net rPMICGPIO1: rU1.8 (GPIO1)
- no-connect marks 24 -> 26
Other:
- note added: "Battery and NTC"
- note removed: "Battery and NTC 10k R4 to simulate "OK" temps"
- moved on the sheet: C2, D24, J2, R4, U1B, U1D, U1H, rC2, rD24, rJ2, rR4, rU1B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

Commit message: add ft200xd, eeprom, and esd protection
Parts:
- added C24, C25, rC24, rC25: 47p, Alidade:C_0603_1608Metric, symbol Alidade:C
- added C26, C28, rC26, rC28: 100n, symbol Alidade:C
- added C27, rC27: 4.7u, symbol Alidade:C
- added R1, R26, rR1, rR26: 27, symbol Alidade:R
- added U5, rU5: FT200XD, Alidade:DFN-10_FTD, symbol Alidade:FT200XD
- added U6, rU6: USBLC6-2SC6, Alidade:SOT23-6L_STM, symbol Alidade:USBLC6-2SC6
- C1: footprint Alidade:C_0603_1608Metric -> (none); LCSC Part # C15849 -> (none)
- L1, L2, rL1, rL2: value 2.2uH -> 2.2u
Connections:
- net DVDD: now also C26.1, U5.2 (RESET#), U5.7 (VCCIO)
- net GND: now also C1.1, C24.2, C25.2, C26.2, C27.2, C28.2, U5.11 (GND), U5.9 (GND), U6.2 (GND); no longer C1.2
- net SCL: now also U5.6 (SCL)
- net SDA: now also U5.8 (SDA)
- net rDVDD: now also rC26.1, rU5.2 (RESET#), rU5.7 (VCCIO)
- net rGND: now also rC1.1, rC24.2, rC25.2, rC26.2, rC27.2, rC28.2, rU5.11 (GND), rU5.9 (GND), rU6.2 (GND); no longer rC1.2
- net rSCL: now also rU5.6 (SCL)
- net rSDA: now also rU5.8 (SDA)
- net rVBUS: now reaches rJ1.A4 (VBUS), rJ1.A9 (VBUS), rJ1.B4 (VBUS), rJ1.B9 (VBUS), rU1.21 (VBUS)
- net rVBUS: now also rC1.2, rC27.1, rC28.1, rU5.4 (VCC), rU6.5 (VBUS); no longer rC1.1
- net at rJ1.A6 (D+): now also rJ1.B6 (D+), rU6.3 (I/O2)
- net at rJ1.A7 (D-): now also rJ1.B7 (D-), rU6.1 (I/O1)
- net VBUS: now reaches J1.A4 (VBUS), J1.A9 (VBUS), J1.B4 (VBUS), J1.B9 (VBUS), U1.21 (VBUS)
- net VBUS: now also C1.2, C27.1, C28.1, U5.4 (VCC), U6.5 (VBUS); no longer C1.1
- net at J1.A6 (D+): now also J1.B6 (D+), U6.3 (I/O2)
- net at J1.A7 (D-): now also J1.B7 (D-), U6.1 (I/O1)
- new net: R26.1, U6.4 (I/O2)
- new net: R1.1, U6.6 (I/O1)
- new net: rC25.1, rR1.2, rU5.1 (USBDM)
- new net: rC24.1, rR26.2, rU5.10 (USBDP)
- new net: rR1.1, rU6.6 (I/O1)
- new net: C25.1, R1.2, U5.1 (USBDM)
- new net: C24.1, R26.2, U5.10 (USBDP)
- new net: rR26.1, rU6.4 (I/O2)
- new net CBUS0: U5.5 (CBUS0)
- new net rCBUS0: rU5.5 (CBUS0)
- no-connect marks 26 -> 20
Other:
- note added: "Type-C Power Input and FTDI"
- note removed: "Type-C Power Input"
- moved on the sheet: C2, C3, C4, C5, C6, D24, J1, J2, R4, U1A, U1B, U1C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

Commit message: Place ftdi parts
Parts:
- C1, C26, C27, C28, rC26, rC27, rC28: footprint (none) -> Alidade:C_0603_1608Metric
- R1, R26, rR1, rR26: footprint (none) -> Alidade:R_0603_1608Metric
Connections:
- net at rJ1.A6 (D+), rJ1.B6 (D+): now also rU6.4 (I/O2); no longer rU6.3 (I/O2)
- net at rJ1.A7 (D-), rJ1.B7 (D-): now also rU6.6 (I/O1); no longer rU6.1 (I/O1)
- net at rR1.1: now also rU6.1 (I/O1); no longer rU6.6 (I/O1)
- net at rR26.1: now also rU6.3 (I/O2); no longer rU6.4 (I/O2)
Other:
- moved on the sheet: rC24, rC25, rR1, rR26, rU5A, rU6
