File: hw/alidade.kicad_pcb (KiCad board)
At the start: 2 copper layers, 277.2 x 107.5 mm, 48 parts, among them J1 TYPE-C-31-M-13C, SW1 SW_Push, SW10 SW_Push, SW11 SW_Push, SW12 SW_Push, SW13 SW_Push, SW14 SW_Push, SW15 SW_Push, SW16 SW_Push, SW17 SW_Push, SW18 SW_Push, SW19 SW_Push, SW2 SW_Push, SW20 SW_Push, SW21 SW_Push, SW3 SW_Push, SW4 SW_Push, SW5 SW_Push, SW6 SW_Push, SW7 SW_Push, SW8 SW_Push, SW9 SW_Push

Commit message: Various footprint updates
Connections:
- net /Power/VBUS renamed Net-(U1C-VBUS)
- net Net-(rJ1-VBUS-PadA4) renamed /PMIC/rVBUS
- EXSW1 pad 1: unconnected-(EXSW1-Pad1) -> Net-(D22-A)
- EXSW1 pad 2: unconnected-(EXSW1-Pad2) -> /HID/ROW2
- EXSW2 pad 1: unconnected-(EXSW2-Pad1) -> Net-(D23-A)
- EXSW2 pad 2: unconnected-(EXSW2-Pad2) -> /HID/ROW3
- J1 pad A6: Net-(U2B-D+) -> unconnected-(J1-D+-PadA6)
- J1 pad A7: Net-(U2B-D-) -> unconnected-(J1-D--PadA7)
- J1 pad B6: Net-(U2B-D+) -> unconnected-(J1-D+-PadB6)
- J1 pad B7: Net-(U2B-D-) -> unconnected-(J1-D--PadB7)
- SW1 pad 1: unconnected-(SW1-Pad1) -> /HID/ROW4
- SW1 pad 2: unconnected-(SW1-Pad2) -> Net-(D1-A)
- SW10 pad 1: unconnected-(SW10-Pad1) -> /HID/ROW3
- SW10 pad 2: unconnected-(SW10-Pad2) -> Net-(D10-A)
- SW11 pad 1: unconnected-(SW11-Pad1) -> /HID/ROW2
- SW11 pad 2: unconnected-(SW11-Pad2) -> Net-(D11-A)
- SW12 pad 1: unconnected-(SW12-Pad1) -> /HID/ROW1
- SW12 pad 2: unconnected-(SW12-Pad2) -> Net-(D12-A)
- SW13 pad 1: unconnected-(SW13-Pad1) -> /HID/ROW1
- SW13 pad 2: unconnected-(SW13-Pad2) -> Net-(D13-A)
- SW14 pad 1: unconnected-(SW14-Pad1) -> /HID/ROW2
- SW14 pad 2: unconnected-(SW14-Pad2) -> Net-(D14-A)
- SW15 pad 1: unconnected-(SW15-Pad1) -> /HID/ROW3
- SW15 pad 2: unconnected-(SW15-Pad2) -> Net-(D15-A)
- SW16 pad 1: unconnected-(SW16-Pad1) -> /HID/ROW3
- SW16 pad 2: unconnected-(SW16-Pad2) -> Net-(D16-A)
- SW17 pad 1: unconnected-(SW17-Pad1) -> /HID/ROW2
- SW17 pad 2: unconnected-(SW17-Pad2) -> Net-(D17-A)
- SW18 pad 1: unconnected-(SW18-Pad1) -> /HID/ROW1
- SW18 pad 2: unconnected-(SW18-Pad2) -> Net-(D18-A)
- SW19 pad 1: unconnected-(SW19-Pad1) -> /HID/ROW1
- SW19 pad 2: unconnected-(SW19-Pad2) -> Net-(D19-A)
- SW2 pad 1: unconnected-(SW2-Pad1) -> /HID/ROW3
- SW2 pad 2: unconnected-(SW2-Pad2) -> Net-(D2-A)
- SW20 pad 1: unconnected-(SW20-Pad1) -> /HID/ROW2
- SW20 pad 2: unconnected-(SW20-Pad2) -> Net-(D20-A)
- SW21 pad 1: unconnected-(SW21-Pad1) -> /HID/ROW3
- SW21 pad 2: unconnected-(SW21-Pad2) -> Net-(D21-A)
- SW3 pad 1: unconnected-(SW3-Pad1) -> /HID/ROW2
- SW3 pad 2: unconnected-(SW3-Pad2) -> Net-(D3-A)
- SW4 pad 1: unconnected-(SW4-Pad1) -> /HID/ROW1
- SW4 pad 2: unconnected-(SW4-Pad2) -> Net-(D4-A)
- SW5 pad 1: unconnected-(SW5-Pad1) -> /HID/ROW1
- SW5 pad 2: unconnected-(SW5-Pad2) -> Net-(D5-A)
- SW6 pad 1: unconnected-(SW6-Pad1) -> /HID/ROW2
- SW6 pad 2: unconnected-(SW6-Pad2) -> Net-(D6-A)
- SW7 pad 1: unconnected-(SW7-Pad1) -> /HID/ROW3
- SW7 pad 2: unconnected-(SW7-Pad2) -> Net-(D7-A)
- SW8 pad 1: unconnected-(SW8-Pad1) -> /HID/ROW4
- SW8 pad 2: unconnected-(SW8-Pad2) -> Net-(D8-A)
- SW9 pad 1: unconnected-(SW9-Pad1) -> /HID/ROW4
- SW9 pad 2: unconnected-(SW9-Pad2) -> Net-(D9-A)
- rEXSW1 pad 1: unconnected-(rEXSW1-Pad1) -> Net-(rD22-A)
- rEXSW1 pad 2: unconnected-(rEXSW1-Pad2) -> /HID/rROW2
- rEXSW2 pad 1: unconnected-(rEXSW2-Pad1) -> Net-(rD23-A)
- rEXSW2 pad 2: unconnected-(rEXSW2-Pad2) -> /HID/rROW3
- rJ1 pad A1: Net-(rJ1-GND-PadA1) -> rGND
- rJ1 pad A12: Net-(rJ1-GND-PadA1) -> rGND
- rJ1 pad A5: unconnected-(rJ1-CC1-PadA5) -> Net-(rJ1-CC1)
- rJ1 pad B1: Net-(rJ1-GND-PadA1) -> rGND
- rJ1 pad B12: Net-(rJ1-GND-PadA1) -> rGND
- rJ1 pad B5: unconnected-(rJ1-CC2-PadB5) -> Net-(rJ1-CC2)
- rJ1 pad S1: unconnected-(rJ1-SHIELD-PadS1) -> rGND
- rSW1 pad 1: unconnected-(rSW1-Pad1) -> /HID/rROW4
- rSW1 pad 2: unconnected-(rSW1-Pad2) -> Net-(rD1-A)
- rSW10 pad 1: unconnected-(rSW10-Pad1) -> /HID/rROW3
- rSW10 pad 2: unconnected-(rSW10-Pad2) -> Net-(rD10-A)
- rSW11 pad 1: unconnected-(rSW11-Pad1) -> /HID/rROW2
- rSW11 pad 2: unconnected-(rSW11-Pad2) -> Net-(rD11-A)
- rSW12 pad 1: unconnected-(rSW12-Pad1) -> /HID/rROW1
- rSW12 pad 2: unconnected-(rSW12-Pad2) -> Net-(rD12-A)
- rSW13 pad 1: unconnected-(rSW13-Pad1) -> /HID/rROW1
- rSW13 pad 2: unconnected-(rSW13-Pad2) -> Net-(rD13-A)
- rSW14 pad 1: unconnected-(rSW14-Pad1) -> /HID/rROW2
- rSW14 pad 2: unconnected-(rSW14-Pad2) -> Net-(rD14-A)
- rSW15 pad 1: unconnected-(rSW15-Pad1) -> /HID/rROW3
- rSW15 pad 2: unconnected-(rSW15-Pad2) -> Net-(rD15-A)
- rSW16 pad 1: unconnected-(rSW16-Pad1) -> /HID/rROW3
- rSW16 pad 2: unconnected-(rSW16-Pad2) -> Net-(rD16-A)
- rSW17 pad 1: unconnected-(rSW17-Pad1) -> /HID/rROW2
- rSW17 pad 2: unconnected-(rSW17-Pad2) -> Net-(rD17-A)
- rSW18 pad 1: unconnected-(rSW18-Pad1) -> /HID/rROW1
- rSW18 pad 2: unconnected-(rSW18-Pad2) -> Net-(rD18-A)
- rSW19 pad 1: unconnected-(rSW19-Pad1) -> /HID/rROW1
- rSW19 pad 2: unconnected-(rSW19-Pad2) -> Net-(rD19-A)
- rSW2 pad 1: unconnected-(rSW2-Pad1) -> /HID/rROW3
- rSW2 pad 2: unconnected-(rSW2-Pad2) -> Net-(rD2-A)
- rSW20 pad 1: unconnected-(rSW20-Pad1) -> /HID/rROW2
- rSW20 pad 2: unconnected-(rSW20-Pad2) -> Net-(rD20-A)
- rSW21 pad 1: unconnected-(rSW21-Pad1) -> /HID/rROW3
- rSW21 pad 2: unconnected-(rSW21-Pad2) -> Net-(rD21-A)
- rSW3 pad 1: unconnected-(rSW3-Pad1) -> /HID/rROW2
- rSW3 pad 2: unconnected-(rSW3-Pad2) -> Net-(rD3-A)
- rSW4 pad 1: unconnected-(rSW4-Pad1) -> /HID/rROW1
- rSW4 pad 2: unconnected-(rSW4-Pad2) -> Net-(rD4-A)
- rSW5 pad 1: unconnected-(rSW5-Pad1) -> /HID/rROW1
- rSW5 pad 2: unconnected-(rSW5-Pad2) -> Net-(rD5-A)
- rSW6 pad 1: unconnected-(rSW6-Pad1) -> /HID/rROW2
- rSW6 pad 2: unconnected-(rSW6-Pad2) -> Net-(rD6-A)
- rSW7 pad 1: unconnected-(rSW7-Pad1) -> /HID/rROW3
- rSW7 pad 2: unconnected-(rSW7-Pad2) -> Net-(rD7-A)
- rSW8 pad 1: unconnected-(rSW8-Pad1) -> /HID/rROW4
- rSW8 pad 2: unconnected-(rSW8-Pad2) -> Net-(rD8-A)
- rSW9 pad 1: unconnected-(rSW9-Pad1) -> /HID/rROW4
- rSW9 pad 2: unconnected-(rSW9-Pad2) -> Net-(rD9-A)
Other:
- outline, holes or cut-outs redrawn
- board text removed: "Jumper for LED"
- board text removed: "v4.1.0"
