File: hw/alidade.kicad_pcb (KiCad board)
At the start: 2 copper layers, 277.2 x 107.5 mm, 48 parts, among them J1 TYPE-C-31-M-13C, SW1 SW_Push, SW10 SW_Push, SW11 SW_Push, SW12 SW_Push, SW13 SW_Push, SW14 SW_Push, SW15 SW_Push, SW16 SW_Push, SW17 SW_Push, SW18 SW_Push, SW19 SW_Push, SW2 SW_Push, SW20 SW_Push, SW21 SW_Push, SW3 SW_Push, SW4 SW_Push, SW5 SW_Push, SW6 SW_Push, SW7 SW_Push, SW8 SW_Push, SW9 SW_Push

Commit message: Soldered switches
Parts:
- EXSW1, EXSW2, SW10, SW11, SW12, SW13, SW14, SW15, SW16, SW17, SW18, SW19, SW2, SW20, SW21, SW3, SW4, SW5, SW6, SW7, SW8, SW9, rEXSW1, rEXSW2, rSW10, rSW11, rSW12, rSW13, rSW14, rSW15, rSW16, rSW17, rSW18, rSW19, rSW2, rSW20, rSW21, rSW3, rSW4, rSW5, rSW6, rSW7, rSW8, rSW9: footprint Alidade:keyswitch_cherrymx_hotswap_1u -> Alidade:CherryMX_ChocV2_1u
- SW1, rSW1: footprint Alidade:keyswitch_cherrymx_hotswap_1.5u -> Alidade:CherryMX_ChocV2_1.5u
- moved rEXSW1 10.0 mm to (219.6, 149.7)
- moved rJ1 10.0 mm to (217.6, 133.7)
- moved rSW1 10.0 mm to (224.6, 201.6)
- moved rSW10 10.0 mm to (276.8, 173.5)
- moved rSW13 10.0 mm to (295.8, 137.8)
- moved rSW5 10.0 mm to (257.7, 137.8)
- moved SW13 10.0 mm to (114.8, 137.8)
- moved SW2 10.0 mm to (172.0, 178.2)
- moved SW3 10.0 mm to (172.0, 159.2)
- moved SW4 10.0 mm to (172.0, 140.1)
- moved rEXSW2 10.0 mm to (219.6, 168.7)
- moved rSW11 10.0 mm to (276.8, 154.4)
- moved rSW12 10.0 mm to (276.8, 135.4)
- moved rSW14 10.0 mm to (295.8, 156.8)
- moved rSW15 10.0 mm to (295.8, 175.9)
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Other:
- outline, holes or cut-outs redrawn

Commit message: pmic left
Parts:
- added C1: 1u, Alidade:C_0603_1608Metric, F.Cu at (179.6, 143.3)
- added C2: 2.2u, Alidade:C_0603_1608Metric, F.Cu at (183.8, 145.0)
- added C3: 1u, Alidade:C_0603_1608Metric, F.Cu at (178.5, 144.8)
- added C4: 10u, Alidade:C_0603_1608Metric, F.Cu at (181.5, 155.2)
- added C5: 10u, Alidade:C_0603_1608Metric, F.Cu at (181.5, 144.8)
- added C6: 10u, Alidade:C_0603_1608Metric, F.Cu at (177.3, 154.8)
- added C7: 10u, Alidade:C_0603_1608Metric, F.Cu at (177.3, 153.3)
- added C8: 10u, Alidade:C_0603_1608Metric, F.Cu at (181.5, 153.7)
- added D24: 19-237/R6GHBHC-A01/2T, Alidade:19-237_R6GHBHC-A01_2T, F.Cu at (184.6, 135.6)
- added L1: 2.2uH, Alidade:L_0603_1608Metric, F.Cu at (175.1, 154.0)
- added L2: 2.2uH, Alidade:L_0603_1608Metric, F.Cu at (181.5, 156.7)
- added R2: 47k, Alidade:R_0603_1608Metric, F.Cu at (185.3, 145.0)
- added R3: 0, Alidade:R_0603_1608Metric, F.Cu at (186.8, 145.0)
- added R4: 0, Alidade:R_0603_1608Metric, F.Cu at (184.8, 137.9)
- added U1: NPM1300-QEAA-R, Alidade:QFN32_5X5, F.Cu at (179.3, 149.2)
- turned EXSW1 to 90 degrees
- turned SW3 to 0 degrees
- turned SW4 to -90 degrees
Routing:
- net Net-(D24-B): track 0.00 -> 26.0 mm
- net Net-(J1-CC2): track 0.00 -> 24.9 mm, vias 0 -> 3
- net GND: track 0.00 -> 24.7 mm
- net Net-(U1C-VBUS): track 0.00 -> 22.2 mm, vias 0 -> 2
- net Net-(D24-G): track 0.00 -> 21.7 mm
- net Net-(J1-CC1): track 0.00 -> 21.2 mm, vias 0 -> 3
- net Net-(D24-R): track 0.00 -> 18.5 mm
- net /PMIC/VSYS: track 0.00 -> 18.0 mm, vias 0 -> 4
- net AVDD: track 0.00 -> 11.4 mm, vias 0 -> 2
- net Net-(U1F-VSET2): track 0.00 -> 5.77 mm
- net Net-(U1F-SW2): track 0.00 -> 5.51 mm, vias 0 -> 2
- net Net-(J2-Pin_1): track 0.00 -> 4.80 mm
- net Net-(U1E-VSET1): track 0.00 -> 4.66 mm
- net Net-(U1E-SW1): track 0.00 -> 4.55 mm, vias 0 -> 2
- net DVDD: track 0.00 -> 4.19 mm
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
Commit message: pmic r
Parts:
- added rC1: 1u, Alidade:C_0603_1608Metric, F.Cu at (232.5, 142.6)
- added rC2: 2.2u, Alidade:C_0603_1608Metric, F.Cu at (236.3, 144.1)
- added rC3: 1u, Alidade:C_0603_1608Metric, F.Cu at (231.0, 144.1)
- added rC4: 10u, Alidade:C_0603_1608Metric, F.Cu at (233.7, 154.0)
- added rC5: 10u, Alidade:C_0603_1608Metric, F.Cu at (234.0, 144.1)
- added rC6: 10u, Alidade:C_0603_1608Metric, F.Cu at (229.5, 154.1)
- added rC7: 10u, Alidade:C_0603_1608Metric, F.Cu at (229.5, 152.6)
- added rC8: 10u, Alidade:C_0603_1608Metric, F.Cu at (233.7, 152.5)
- added rD24: 19-237/R6GHBHC-A01/2T, Alidade:19-237_R6GHBHC-A01_2T, F.Cu at (226.6, 136.1)
- added rL1: 2.2uH, Alidade:L_0603_1608Metric, F.Cu at (227.3, 153.3)
- added rL2: 2.2uH, Alidade:L_0603_1608Metric, F.Cu at (233.8, 155.5)
- added rR2: 47k, Alidade:R_0603_1608Metric, F.Cu at (237.8, 144.1)
- added rR3: 0, Alidade:R_0603_1608Metric, F.Cu at (239.3, 144.1)
- added rR4: 0, Alidade:R_0603_1608Metric, F.Cu at (228.3, 138.9)
- added rU1: NPM1300-QEAA-R, Alidade:QFN32_5X5, F.Cu at (231.5, 148.6)
- EXSW1, EXSW2, SW10, SW11, SW12, SW13, SW14, SW15, SW16, SW17, SW18, SW19, SW2, SW20, SW21, SW3, SW4, SW5, SW6, SW7, SW8, SW9, rEXSW1, rEXSW2, rSW10, rSW11, rSW12, rSW13, rSW14, rSW15, rSW16, rSW17, rSW18, rSW19, rSW2, rSW20, rSW21, rSW3, rSW4, rSW5, rSW6, rSW7, rSW8, rSW9: footprint Alidade:CherryMX_ChocV2_1u -> Alidade:CherryMX_1u
- SW1, rSW1: footprint Alidade:CherryMX_ChocV2_1.5u -> Alidade:CherryMX_1u
- moved C4 0.55 mm to (181.5, 154.6)
- moved C8 0.55 mm to (181.5, 153.1)
- moved L2 0.55 mm to (181.5, 156.1)
- turned EXSW1 to 0 degrees
- turned SW11 to 0 degrees
- turned SW14 to 0 degrees
- turned SW17 to 0 degrees
- turned SW20 to 0 degrees
- turned SW6 to 0 degrees
- turned rEXSW1 to 0 degrees
- turned rSW11 to 0 degrees
- turned rSW14 to 0 degrees
- turned rSW17 to 0 degrees
- turned rSW20 to 0 degrees
- turned rSW3 to 0 degrees
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Routing:
- net rGND: track 0.00 -> 25.7 mm
- net /PMIC/rVBUS: track 0.00 -> 22.1 mm, vias 0 -> 2
- net Net-(rJ1-CC1): track 0.00 -> 18.0 mm, vias 0 -> 1
- net /PMIC/rVSYS: track 0.00 -> 17.7 mm, vias 0 -> 2
- net Net-(rD24-G): track 0.00 -> 17.4 mm, vias 0 -> 2
- net Net-(rD24-B): track 0.00 -> 15.0 mm, vias 0 -> 2
- net Net-(rJ1-CC2): track 0.00 -> 14.1 mm, vias 0 -> 1
- net Net-(rD24-R): track 0.00 -> 13.7 mm, vias 0 -> 2
- net rAVDD: track 0.00 -> 11.0 mm, vias 0 -> 2
- net Net-(rU1F-VSET2): track 0.00 -> 6.15 mm
- net Net-(rU1E-VSET1): track 0.00 -> 5.04 mm
- net Net-(rU1F-SW2): track 0.00 -> 4.93 mm, vias 0 -> 2
- net Net-(rJ2-Pin_1): track 0.00 -> 4.92 mm
- net Net-(rD24-Pad4): track 0.00 -> 4.78 mm
- net Net-(rU1E-SW1): track 0.00 -> 4.48 mm, vias 0 -> 2
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
Commit message: Fix silkscreens
Other:
- outline, holes or cut-outs redrawn
- rule pad_to_mask_clearance: 0.2 -> 0.1
Changed lines of the file:
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@@
 			(dielectric_constraints no)
 		)
-		(pad_to_mask_clearance 0.2)
+		(pad_to_mask_clearance 0.1)
 		(allow_soldermask_bridges_in_footprints no)
 		(tenting front back)
@@
 		(at 226.565 136.11125 -90)
 		(property "Reference" "rD24"
-			(at 0.582 -1.6564 90)
+			(at 0 -2 270)
 			(layer "F.SilkS")
 			(effects
 				(font
-					(size 0.64 0.64)
+					(size 1 1)
 					(thickness 0.15)
 				)
@@
 		(tags "resistor")
 		(property "Reference" "rR4"
-			(at 0 -1.43 0)
+			(at 0 1.5 0)
 			(layer "F.SilkS")
 			(effects
@@
 		(tags "resistor")
 		(property "Reference" "R4"
-			(at 0 -1.43 0)
+			(at 0 1.5 0)
 			(layer "F.SilkS")
 			(effects
@@
 		(tags "NPM1300-QEAA-R7 ")
 		(property "Reference" "rU1"
-			(at 0 0 90)
+			(at 0.25 -3.974999 90)
 			(unlocked yes)
 			(layer "F.SilkS")
@@
 		(tags "capacitor")
 		(property "Reference" "rC8"
-			(at 0 -1.43 0)
+			(at -2.824301 0.112001 0)
 			(layer "F.SilkS")
 			(effects
@@
 		(tags "capacitor")
 		(property "Reference" "rC6"
-			(at 0 -1.43 0)
+			(at -0.049301 -2.749999 0)
 			(layer "F.SilkS")
 			(effects
@@
 		(tags "resistor")
 		(property "Reference" "rR2"
-			(at 0 -1.43 90)
+			(at 2.75 0 90)
 			(layer "F.SilkS")
 			(effects
@@
 		(tags "capacitor")
 		(property "Reference" "rC7"
-			(at 0 -1.43 0)
+			(at 0 2.999999 0)
 			(layer "F.SilkS")
 			(effects
@@
 		(tags "capacitor")
 		(property "Reference" "rC5"
-			(at 2.75 0 0)
+			(at 1.275 -2.25 0)
 			(layer "F.SilkS")
 			(effects
@@
 		(tags "inductor")
 		(property "Reference" "rL2"
-			(at 0 -1.43 0)
+			(at -2.799301 0.112001 0)
 			(layer "F.SilkS")
 			(effects
@@
 		(tags "capacitor")
 		(property "Reference" "rC4"
-			(at 0 -1.43 0)
+			(at 2.824301 -0.112001 0)
 			(layer "F.SilkS")
 			(effects
@@
 		(tags "resistor")
 		(property "Reference" "rR3"
-			(at 0 -1.43 90)
+			(at 2.75 0 90)
 			(layer "F.SilkS")
 			(effects
@@
 		(tags "capacitor")
 		(property "Reference" "rC2"
-			(at 0 -1.43 90)
+			(at -2.75 0 90)
 			(layer "F.SilkS")
 			(effects
@@
 		(at 184.565 135.61125 -90)
 		(property "Reference" "D24"
-			(at 0.582 -1.6564 90)
+			(at 0 1.75 90)
 			(layer "F.SilkS")
 			(effects
 				(font
-					(size 0.64 0.64)
+					(size 1 1)
 					(thickness 0.15)
 				)
@@
 		(layer "Edge.Cuts")
 	)
-	(gr_circle
-		(center 248.177502 148.483125)
-		(end 245.677502 148.483125)
-		(stroke
-			(width 0.1)
-			(type solid)
-		)
-		(fill no)
-		(layer "Edge.Cuts")
-	)
 	(gr_curve
 		(pts
@@
 		(layer "Edge.Cuts")
 	)
-	(gr_circle
-		(center 307.232502 152.055)
-		(end 304.732502 152.055)
-		(stroke
-			(width 0.1)
-			(type solid)
-		)
-		(fill no)
-		(layer "Edge.Cuts")
-	)
 	(gr_curve
 		(pts
@@
 		(layer "Edge.Cuts")
 	)
-	(gr_circle
-		(center 162.4525 148.483125)
-		(end 164.9525 148.483125)
-		(stroke
-			(width 0.1)
-			(type solid)
-		)
-		(fill no)
-		(layer "Edge.Cuts")
-	)
 	(gr_line
 		(start 67.702498 190.655)
@@
 		(layer "Edge.Cuts")
 	)
-	(gr_circle
-		(center 103.3975 171.105)
-		(end 105.8975 171.105)
-		(stroke
-			(width 0.1)
-			(type solid)
-		)
-		(fill no)
-		(layer "Edge.Cuts")
-	)
 	(gr_curve
 		(pts
@@
 		(layer "Edge.Cuts")
 	)
-	(gr_circle
-		(center 86.2525 152.055)
-		(end 88.7525 152.055)
-		(stroke
-			(width 0.1)
-			(type solid)
-		)
-		(fill no)
-		(layer "Edge.Cuts")
-	)
 	(gr_line
 		(start 312.4775 190.655)
@@
 		(layer "Edge.Cuts")
 	)
-	(gr_circle
-		(center 307.232502 171.105)
-		(end 304.732502 171.105)
-		(stroke
-			(width 0.1)
-			(type solid)
-		)
-		(fill no)
-		(layer "Edge.Cuts")
-	)
 	(gr_curve
 		(pts
@@
 		(layer "Edge.Cuts")
 	)
-	(gr_circle
-		(center 324.377502 152.055)
-		(end 321.877502 152.055)
-		(stroke
-			(width 0.1)
-			(type solid)
-		)
-		(fill no)
-		(layer "Edge.Cuts")
-	)
 	(gr_curve
 		(pts
@@
 		(layer "Edge.Cuts")
 	)
-	(gr_circle
-		(center 103.3975 152.055)
-		(end 105.8975 152.055)
-		(stroke
-			(width 0.1)
-			(type solid)
-		)
-		(fill no)
-		(layer "Edge.Cuts")
-	)
 	(gr_curve
 		(pts
@@
 		(layer "Edge.Cuts")
 	)
-	(gr_circle
-		(center 324.377502 171.105)
-		(end 321.877502 171.105)
-		(stroke
-			(width 0.1)
-			(type solid)
-		)
-		(fill no)
-		(layer "Edge.Cuts")
-	)
 	(gr_curve
 		(pts
@@
 		(layer "Edge.Cuts")
 	)
-	(gr_circle
-		(center 162.452498 187.77375)
-		(end 164.952498 187.77375)
-		(stroke
-			(width 0.1)
-			(type solid)
-		)
-		(fill no)
-		(layer "Edge.Cuts")
-	)
 	(gr_curve
 		(pts
@@
 		(layer "Edge.Cuts")
 	)
-	(gr_circle
-		(center 86.2525 171.105)
-		(end 88.7525 171.105)
-		(stroke
-			(width 0.1)
-			(type solid)
-		)
-		(fill no)
-		(layer "Edge.Cuts")
-	)
 	(gr_curve
 		(pts
@@
 		(layer "Edge.Cuts")
 	)
-	(gr_circle
-		(center 248.177504 187.77375)
-		(end 245.677504 187.77375)
-		(stroke
-			(width 0.1)
-			(type solid)
-		)
-		(fill no)
-		(layer "Edge.Cuts")
-	)
 	(gr_line
 		(start 336.2775 190.655)
@@
 	)
 	(gr_line
-		(start 188.9846 218.4768)
-		(end 200.5525 192.348)
-		(stroke
-			(width 0.1)
-			(type default)
-		)
-		(layer "F.Fab")
-	)
-	(gr_line
 		(start 105.3025 128.2425)
 		(end 124.3525 128.2425)
@@
 	)
 	(gr_line
-		(start 67.2025 190.155)
-		(end 124.3525 190.155)
-		(stroke
-			(width 0.1)
-			(type default)
-		)
-		(layer "F.Fab")
-	)
-	(gr_line
 		(start 124.3525 125.86125)
 		(end 143.4025 125.86125)
@@
 	)
 	(gr_line
-		(start 133.8775 206.82375)
-		(end 171.5653 210.765)
-		(stroke
-			(width 0.1)
-			(type default)
-		)
-		(layer "F.Fab")
-	)
-	(gr_line
-		(start 171.5653 210.765)
-		(end 188.9846 218.4768)
-		(stroke
-			(width 0.1)
-			(type default)
-		)
-		(layer "F.Fab")
-	)
-	(gr_line
 		(start 143.4025 125.86125)
 		(end 143.4025 128.2425)
 		(stroke
 			(width 0.1)
-			(type default)
-		)
-		(layer "F.Fab")
-	)
-	(gr_line
-		(start 124.3525 190.155)
-		(end 133.8775 206.82375)
-		(stroke
-			(width 0.1)

Commit message: mcu l
Parts:
- added ANT1: SWRA117D, Alidade:Texas_SWRA117D_2.4GHz_Left, F.Cu at (195.2, 189.4)
- added C12: 100n, Alidade:C_0603_1608Metric, F.Cu at (179.8, 181.0)
- added C13: 100n, Alidade:C_0603_1608Metric, F.Cu at (182.2, 174.0)
- added C14: 100n, Alidade:C_0603_1608Metric, F.Cu at (190.4, 182.9)
- added C15: 100n, Alidade:C_0603_1608Metric, F.Cu at (189.5, 176.4)
- added C16: 10u, Alidade:C_0603_1608Metric, F.Cu at (189.5, 174.9)
- added C17: 2.2u, Alidade:C_0603_1608Metric, F.Cu at (191.8, 175.9)
- added C18: 2.2u, Alidade:C_0603_1608Metric, F.Cu at (184.6, 185.9)
- added C19: 10n, Alidade:C_0603_1608Metric, F.Cu at (190.1, 179.1)
- added C20: 2.2n, Alidade:C_0603_1608Metric, F.Cu at (184.6, 184.4)
- added C21: 0.3p, Alidade:C_0603_1608Metric, F.Cu at (194.1, 191.6)
- added C22: 2p, Alidade:C_0603_1608Metric, F.Cu at (191.8, 191.6)
- added C23: 1.5p, Alidade:C_0603_1608Metric, F.Cu at (188.0, 187.9)
- added FB1: FB, Alidade:L_0603_1608Metric, F.Cu at (193.1, 179.1)
- added L3: 4.7u, Alidade:L_0603_1608Metric, F.Cu at (193.3, 175.9)
- added L4: 3.5n, Alidade:L_0603_1608Metric, F.Cu at (193.3, 189.4)
- added L5: 3.5n, Alidade:L_0603_1608Metric, F.Cu at (190.3, 189.4)
- added L6: 2.7n, Alidade:L_0603_1608Metric, F.Cu at (187.3, 189.4)
- added U2: NRF54L15-QFAA-R, Alidade:QFN48_6X6, F.Cu at (184.4, 178.8)
- added Y1: ABS07-32.768KHZ-T, Alidade:XTAL_ABS07-32.768KHZ-1-T, F.Cu at (186.7, 173.2)
- added Y2: ABM8G-32.000MHZ-B4Y-T, Alidade:XTAL_ABM8G-32.000MHZ-B4Y-T, F.Cu at (187.9, 184.5)
Routing:
- net Net-(U2F-DECA): track 0.00 -> 26.5 mm, vias 0 -> 5
- net GND: track 26.4 -> 47.7 mm
- net DVDD: track 4.19 -> 16.5 mm
- net Net-(U2F-DECD): track 0.00 -> 9.25 mm
- net Net-(U2E-ANT): track 0.00 -> 8.43 mm
- net Net-(U2F-DCC): track 0.00 -> 6.30 mm, vias 0 -> 2
- net Net-(U2E-XC1): track 0.00 -> 6.07 mm
- net Net-(U2B-P1.00/XL1): track 0.00 -> 5.41 mm
- net Net-(C23-Pad1): track 0.00 -> 2.91 mm
- net Net-(C22-Pad1): track 0.00 -> 2.88 mm
- net Net-(ANT1-FEED): track 0.00 -> 2.57 mm
- net Net-(U2E-XC2): track 0.00 -> 2.04 mm
- net Net-(U2B-P1.01/XL2): track 0.00 -> 1.62 mm
- net /HID/ROW4: track 0.00 -> 0.96 mm, vias 0 -> 1
Other:
- rule pad_to_mask_clearance: 0.1 -> 0.05

Commit message: mcu r
Parts:
- added rANT1: SWRA117D, Alidade:Texas_SWRA117D_2.4GHz_Right, F.Cu at (215.4, 189.4)
- added rC12: 100n, Alidade:C_0603_1608Metric, F.Cu at (216.6, 180.9)
- added rC13: 100n, Alidade:C_0603_1608Metric, F.Cu at (219.0, 173.9)
- added rC14: 100n, Alidade:C_0603_1608Metric, F.Cu at (227.2, 182.7)
- added rC15: 100n, Alidade:C_0603_1608Metric, F.Cu at (226.3, 176.3)
- added rC16: 10u, Alidade:C_0603_1608Metric, F.Cu at (226.3, 174.8)
- added rC17: 2.2u, Alidade:C_0603_1608Metric, F.Cu at (228.5, 176.0)
- added rC18: 2.2u, Alidade:C_0603_1608Metric, F.Cu at (221.4, 185.9)
- added rC19: 10n, Alidade:C_0603_1608Metric, F.Cu at (226.9, 178.8)
- added rC20: 2.2n, Alidade:C_0603_1608Metric, F.Cu at (221.4, 184.4)
- added rC21: 0.3p, Alidade:C_0603_1608Metric, F.Cu at (216.6, 191.6)
- added rC22: 2p, Alidade:C_0603_1608Metric, F.Cu at (218.8, 191.6)
- added rC23: 1.5p, Alidade:C_0603_1608Metric, F.Cu at (222.6, 187.9)
- added rFB1: FB, Alidade:L_0603_1608Metric, F.Cu at (229.9, 178.8)
- added rL3: 4.7u, Alidade:L_0603_1608Metric, F.Cu at (230.0, 176.0)
- added rL4: 3.5n, Alidade:L_0603_1608Metric, F.Cu at (217.3, 189.4)
- added rL5: 3.5n, Alidade:L_0603_1608Metric, F.Cu at (220.3, 189.4)
- added rL6: 2.7n, Alidade:L_0603_1608Metric, F.Cu at (223.3, 189.4)
- added rU4: NRF54L15-QFAA-R, Alidade:QFN48_6X6, F.Cu at (221.2, 178.7)
- added rY1: ABS07-32.768KHZ-T, Alidade:XTAL_ABS07-32.768KHZ-1-T, F.Cu at (223.4, 173.0)
- added rY2: ABM8G-32.000MHZ-B4Y-T, Alidade:XTAL_ABM8G-32.000MHZ-B4Y-T, F.Cu at (224.8, 184.4)
- moved J1 0.10 mm to (193.0, 133.8)
- moved rJ1 0.10 mm to (217.6, 133.8)
Routing:
- net rGND: track 25.7 -> 46.8 mm
- net Net-(rU4F-DECA): track 0.00 -> 20.3 mm, vias 0 -> 3
- net rDVDD: track 4.14 -> 16.3 mm
- net Net-(rU4F-DECD): track 0.00 -> 10.5 mm
- net Net-(rU4E-ANT): track 0.00 -> 9.18 mm
- net Net-(rU4F-DCC): track 0.00 -> 6.34 mm, vias 0 -> 2
- net Net-(rU4E-XC1): track 0.00 -> 5.86 mm
- net Net-(rU4B-P1.00/XL1): track 0.00 -> 5.27 mm
- net Net-(rC23-Pad1): track 0.00 -> 2.94 mm
- net Net-(rC22-Pad1): track 0.00 -> 2.91 mm
- net Net-(rANT1-FEED): track 0.00 -> 2.60 mm
- net Net-(rU4E-XC2): track 0.00 -> 2.05 mm
- net Net-(rU4B-P1.01/XL2): track 0.00 -> 1.69 mm
- net /HID/ROW4: track 0.96 -> 0.00 mm, vias 1 -> 0

Commit message: trackpoint l
Parts:
- added C10: 100n, Alidade:C_0603_1608Metric, F.Cu at (149.2, 154.7)
- added C11: 100n, Alidade:C_0603_1608Metric, F.Cu at (149.2, 153.2)
- added C9: 100n, Alidade:C_0603_1608Metric, F.Cu at (145.7, 153.2)
- added M1: SK8701-01-005-SENSOR, Alidade:SK8707-01-005-SENSOR, F.Cu at (162.5, 148.5)
- added R15: 2.4k, Alidade:R_0603_1608Metric, F.Cu at (153.7, 143.3)
- added R16: 2.4k, Alidade:R_0603_1608Metric, F.Cu at (152.2, 143.3)
- added R17: 0, Alidade:R_0603_1608Metric, F.Cu at (180.0, 175.0)
- added R18: 0, Alidade:R_0603_1608Metric, F.Cu at (178.1, 175.0)
- added U3: ADS122S14IRTER, Alidade:WQFN16_3X3, F.Cu at (147.5, 150.7)
- moved C13 0.07 mm to (182.3, 174.0)
- turned SW4 to 180 degrees
Connections:
- net /PMIC/rVBUS renamed Net-(rU1C-VBUS)
Routing:
- net /HID/FAULT: track 0.00 -> 60.8 mm, vias 0 -> 2
- net /HID/DRDY: track 0.00 -> 58.8 mm, vias 0 -> 2
- net /HID/ADCCS: track 0.00 -> 56.8 mm
- net /HID/MISO: track 0.00 -> 55.7 mm, vias 0 -> 2
- net /HID/SCK: track 0.00 -> 49.8 mm
- net /HID/MOSI: track 0.00 -> 48.5 mm
- net Net-(U3A-AIN1): track 0.00 -> 15.3 mm
- net /HID/REFP: track 0.00 -> 8.88 mm
- net /HID/REFN: track 0.00 -> 7.75 mm
- net Net-(U2C-P2.04/SPI.SDI/SDO): track 0.00 -> 4.35 mm
- net AVDD: track 10.9 -> 13.7 mm
- net Net-(D24-B): track 26.0 -> 28.6 mm
- net /HID/AIN0: track 0.00 -> 2.57 mm
- net /HID/AIN1: track 0.00 -> 2.25 mm
- net Net-(U2C-P2.01/SPI.SCK): track 0.00 -> 2.19 mm
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
Commit message: trackpoint r
Parts:
- added rC10: 100n, Alidade:C_0603_1608Metric, F.Cu at (261.4, 142.3)
- added rC11: 100n, Alidade:C_0603_1608Metric, F.Cu at (261.4, 143.8)
- added rC9: 100n, Alidade:C_0603_1608Metric, F.Cu at (265.4, 143.8)
- added rM2: SK8701-01-005-SENSOR, Alidade:SK8707-01-005-SENSOR, F.Cu at (248.2, 148.5)
- added rR15: 2.4k, Alidade:R_0603_1608Metric, F.Cu at (257.9, 143.2)
- added rR16: 2.4k, Alidade:R_0603_1608Metric, F.Cu at (256.4, 143.2)
- added rR17: 0, Alidade:R_0603_1608Metric, F.Cu at (216.7, 174.7)
- added rR18: 0, Alidade:R_0603_1608Metric, F.Cu at (214.9, 174.7)
- added rU3: ADS122S14IRTER, Alidade:WQFN16_3X3, F.Cu at (263.5, 146.3)
- moved rY1 0.05 mm to (223.4, 173.0)
Routing:
- net /HID/rADCCS: track 0.00 -> 91.0 mm
- net /HID/rMISO: track 0.00 -> 87.9 mm, vias 0 -> 2
- net /HID/rDRDY: track 0.00 -> 87.0 mm, vias 0 -> 2
- net /HID/rMOSI: track 0.00 -> 86.2 mm
- net /HID/rSCK: track 0.00 -> 70.7 mm
- net /HID/rFAULT: track 0.00 -> 66.1 mm, vias 0 -> 4
- net /HID/rREFN: track 0.00 -> 13.4 mm
- net /HID/rREFP: track 0.00 -> 10.2 mm
- net Net-(rU3A-AIN1): track 0.00 -> 7.65 mm
- net Net-(rU4C-P2.04/SPI.SDI/SDO): track 0.00 -> 4.28 mm
- net rAVDD: track 11.0 -> 14.1 mm
- net /HID/rAIN0: track 0.00 -> 2.96 mm
- net /HID/rAIN1: track 0.00 -> 2.64 mm
- net Net-(rU4C-P2.01/SPI.SCK): track 0.00 -> 2.41 mm
- net Net-(rU3C-REFOUT): track 0.00 -> 1.40 mm
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