File: hw/alidade.kicad_pcb (KiCad board)
At the start: 2 copper layers, 277.2 x 107.5 mm, 138 parts, among them J1 TYPE-C-31-M-13C, M1 SK8701-01-005-SENSOR, SW1 SW_Push, SW10 SW_Push, SW11 SW_Push, SW12 SW_Push, SW13 SW_Push, SW14 SW_Push, SW15 SW_Push, SW16 SW_Push, SW17 SW_Push, SW18 SW_Push, SW19 SW_Push, SW2 SW_Push, SW20 SW_Push, SW21 SW_Push, SW3 SW_Push, SW4 SW_Push, SW5 SW_Push, SW6 SW_Push, SW7 SW_Push, SW8 SW_Push, SW9 SW_Push, U1 NPM1300-QEAA-R, U2 NRF54L15-QFAA-R, U3 ADS122S14IRTER, Y1 ABS07-32.768KHZ-T, Y2 ABM8G-32.000MHZ-B4Y-T

Commit message: Diodes left
Parts:
- added D1: BAT54, Alidade:SOT23, F.Cu at (181.1, 198.1)
- added D10: BAT54, Alidade:SOT23, F.Cu at (135.1, 167.5)
- added D11: BAT54, Alidade:SOT23, F.Cu at (132.7, 160.4)
- added D12: BAT54, Alidade:SOT23, F.Cu at (135.1, 129.4)
- added D13: BAT54, Alidade:SOT23, F.Cu at (116.0, 131.8)
- added D14: BAT54, Alidade:SOT23, F.Cu at (113.6, 162.8)
- added D15: BAT54, Alidade:SOT23, F.Cu at (116.0, 169.9)
- added D16: BAT54, Alidade:SOT23, F.Cu at (97.0, 174.6)
- added D17: BAT54, Alidade:SOT23, F.Cu at (94.6, 167.5)
- added D18: BAT54, Alidade:SOT23, F.Cu at (97.0, 136.5)
- added D19: BAT54, Alidade:SOT23, F.Cu at (77.9, 136.6)
- added D2: BAT54, Alidade:SOT23, F.Cu at (173.2, 172.3)
- added D20: BAT54, Alidade:SOT23, F.Cu at (75.5, 167.5)
- added D21: BAT54, Alidade:SOT23, F.Cu at (77.9, 174.7)
- added D22: BAT54, Alidade:SOT23, F.Cu at (189.8, 155.6)
- added D23: BAT54, Alidade:SOT23, F.Cu at (192.2, 162.8)
- added D3: BAT54, Alidade:SOT23, F.Cu at (170.8, 165.2)
- added D4: BAT54, Alidade:SOT23, F.Cu at (173.2, 134.2)
- added D5: BAT54, Alidade:SOT23, F.Cu at (154.1, 131.8)
- added D6: BAT54, Alidade:SOT23, F.Cu at (151.7, 162.8)
- added D7: BAT54, Alidade:SOT23, F.Cu at (154.1, 169.9)
- added D8: BAT54, Alidade:SOT23, F.Cu at (166.6, 193.9)
- added D9: BAT54, Alidade:SOT23, F.Cu at (144.6, 191.3)
Connections:
- EXSW1 pad 1: Net-(D22-A) -> /HID/ROW2
- EXSW1 pad 2: /HID/ROW2 -> Net-(D22-A)
- EXSW2 pad 1: Net-(D23-A) -> /HID/ROW3
- EXSW2 pad 2: /HID/ROW3 -> Net-(D23-A)
Routing:
- net /HID/ROW2: track 0.00 -> 124.1 mm, vias 0 -> 2
- net /HID/ROW3: track 0.00 -> 100.2 mm
- net /HID/ROW1: track 0.00 -> 100.2 mm
- net /HID/COL2: track 0.00 -> 72.3 mm, vias 0 -> 10
- net /HID/COL3: track 0.00 -> 72.1 mm, vias 0 -> 8
- net /HID/COL4: track 0.00 -> 70.3 mm, vias 0 -> 6
- net /HID/COL6: track 0.00 -> 42.3 mm, vias 0 -> 4
- net /HID/COL5: track 0.00 -> 42.3 mm, vias 0 -> 4
- net /HID/COL7: track 0.00 -> 42.2 mm, vias 0 -> 2
- net /HID/ROW4: track 0.00 -> 40.9 mm
- net /HID/COL1: track 0.00 -> 6.41 mm
- net /HID/MOSI: track 48.5 -> 53.1 mm
- net /HID/ADCCS: track 56.8 -> 61.3 mm
- net /HID/DRDY: track 58.8 -> 62.4 mm
- net /HID/SCK: track 49.8 -> 53.3 mm
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
Commit message: Diodes right
Parts:
- added rD1: BAT54, Alidade:SOT23, F.Cu at (230.5, 200.2)
- added rD10: BAT54, Alidade:SOT23, F.Cu at (278.0, 167.5)
- added rD11: BAT54, Alidade:SOT23, F.Cu at (275.6, 160.4)
- added rD12: BAT54, Alidade:SOT23, F.Cu at (277.9, 129.4)
- added rD13: BAT54, Alidade:SOT23, F.Cu at (297.0, 131.8)
- added rD14: BAT54, Alidade:SOT23, F.Cu at (294.6, 162.8)
- added rD15: BAT54, Alidade:SOT23, F.Cu at (297.0, 169.9)
- added rD16: BAT54, Alidade:SOT23, F.Cu at (316.0, 174.7)
- added rD17: BAT54, Alidade:SOT23, F.Cu at (313.7, 167.5)
- added rD18: BAT54, Alidade:SOT23, F.Cu at (316.0, 136.5)
- added rD19: BAT54, Alidade:SOT23, F.Cu at (335.1, 136.6)
- added rD2: BAT54, Alidade:SOT23, F.Cu at (239.9, 172.3)
- added rD20: BAT54, Alidade:SOT23, F.Cu at (332.7, 167.5)
- added rD21: BAT54, Alidade:SOT23, F.Cu at (335.1, 174.7)
- added rD22: BAT54, Alidade:SOT23, F.Cu at (218.4, 155.6)
- added rD23: BAT54, Alidade:SOT23, F.Cu at (220.8, 162.8)
- added rD3: BAT54, Alidade:SOT23, F.Cu at (237.5, 165.1)
- added rD4: BAT54, Alidade:SOT23, F.Cu at (239.8, 134.2)
- added rD5: BAT54, Alidade:SOT23, F.Cu at (258.9, 131.8)
- added rD6: BAT54, Alidade:SOT23, F.Cu at (256.5, 162.8)
- added rD7: BAT54, Alidade:SOT23, F.Cu at (258.9, 169.9)
- added rD8: BAT54, Alidade:SOT23, F.Cu at (246.4, 193.4)
- added rD9: BAT54, Alidade:SOT23, F.Cu at (268.4, 191.3)
- moved Y1 0.10 mm to (186.6, 173.2)
Connections:
- rEXSW1 pad 1: Net-(rD22-A) -> /HID/rROW2
- rEXSW1 pad 2: /HID/rROW2 -> Net-(rD22-A)
- rEXSW2 pad 1: Net-(rD23-A) -> /HID/rROW3
- rEXSW2 pad 2: /HID/rROW3 -> Net-(rD23-A)
Routing:
- net /HID/rROW2: track 0.00 -> 126.3 mm, vias 0 -> 2
- net /HID/rROW3: track 0.00 -> 100.2 mm
- net /HID/rROW1: track 0.00 -> 100.2 mm
- net /HID/rCOL2: track 0.00 -> 76.8 mm, vias 0 -> 4
- net /HID/rCOL3: track 0.00 -> 74.7 mm, vias 0 -> 8
- net /HID/rCOL4: track 0.00 -> 71.7 mm, vias 0 -> 6
- net /HID/rROW4: track 0.00 -> 46.4 mm
- net /HID/rCOL7: track 0.00 -> 42.7 mm, vias 0 -> 2
- net /HID/rCOL6: track 0.00 -> 42.6 mm, vias 0 -> 4
- net /HID/rCOL5: track 0.00 -> 42.4 mm, vias 0 -> 4
- net /HID/rCOL1: track 0.00 -> 7.44 mm, vias 0 -> 2
- net Net-(rD1-A): track 0.00 -> 3.02 mm
- net Net-(rD8-A): track 0.00 -> 2.96 mm
- net Net-(rD5-A): track 0.00 -> 2.84 mm
- net Net-(rD6-A): track 0.00 -> 2.84 mm
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
Commit message: shphld switches
Parts:
- added R11: 10k, Alidade:R_0603_1608Metric, F.Cu at (130.0, 178.1)
- added R12: 10k, Alidade:R_0603_1608Metric, F.Cu at (132.6, 179.6)
- added R13: 0, Alidade:R_0603_1608Metric, F.Cu at (130.7, 176.8)
- added R14: 0, Alidade:R_0603_1608Metric, F.Cu at (133.3, 178.3)
- added SWD1: 228ADS2AAWFCMBA, Alidade:228ADS2, F.Cu at (130.5, 184.0)
- added rR11: 10k, Alidade:R_0603_1608Metric, F.Cu at (278.4, 179.4)
- added rR12: 10k, Alidade:R_0603_1608Metric, F.Cu at (281.0, 177.9)
- added rR13: 0, Alidade:R_0603_1608Metric, F.Cu at (277.7, 178.1)
- added rR14: 0, Alidade:R_0603_1608Metric, F.Cu at (280.2, 176.6)
- added rSWD1: 228ADS2AAWFCMBA, Alidade:228ADS2, F.Cu at (284.0, 181.8)
Routing:
- net Net-(rR11-Pad2): track 0.00 -> 9.65 mm
- net Net-(R11-Pad2): track 0.00 -> 9.62 mm
- net Net-(R12-Pad1): track 0.00 -> 9.60 mm
- net Net-(rR12-Pad2): track 0.00 -> 9.40 mm
- net GND: track 48.0 -> 54.8 mm
- net rGND: track 46.8 -> 53.5 mm
- net /HID/SHPHLD: track 0.00 -> 5.37 mm
- net /HID/rSHPHLD: track 0.00 -> 5.36 mm
- net rDVDD: track 17.6 -> 19.0 mm
- net DVDD: track 17.6 -> 19.1 mm
- net /HID/rCOL7: track 42.7 -> 43.4 mm
