File: hw/hid.kicad_sch (KiCad schematic)
At the start: 124 parts, among them M1 SK8701-01-005-SENSOR, SW1 SW_Push, SW10 SW_Push, SW11 SW_Push, SW12 SW_Push, SW13 SW_Push, SW14 SW_Push, SW15 SW_Push, SW16 SW_Push, SW17 SW_Push, SW18 SW_Push, SW19 SW_Push, SW2 SW_Push, SW20 SW_Push, SW21 SW_Push, SW3 SW_Push, SW4 SW_Push, SW5 SW_Push, SW6 SW_Push, SW7 SW_Push, SW8 SW_Push, SW9 SW_Push, U3 ADS122S14IRTER

Commit message: Place ftdi parts
Connections:
- net ROW2: now also EXSW1.1; no longer EXSW1.2
- net ROW3: now also EXSW2.1; no longer EXSW2.2
- net rROW2: now also rEXSW1.1; no longer rEXSW1.2
- net rROW3: now also rEXSW2.1; no longer rEXSW2.2
- net at D23.1 (A): now also EXSW2.2; no longer EXSW2.1
- net at D22.1 (A): now also EXSW1.2; no longer EXSW1.1
- net at rD23.1 (A): now also rEXSW2.2; no longer rEXSW2.1
- net at rD22.1 (A): now also rEXSW1.2; no longer rEXSW1.1
Changed lines of the file:
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@@
 		(lib_id "Alidade:SW_Push")
 		(at 172.72 97.79 0)
-		(mirror y)
 		(unit 1)
 		(body_style 1)
@@
 		(lib_id "Alidade:SW_Push")
 		(at 172.72 82.55 0)
-		(mirror y)
 		(unit 1)
 		(body_style 1)
@@
 		(lib_id "Alidade:SW_Push")
 		(at 248.92 97.79 0)
+		(mirror y)
 		(unit 1)
 		(body_style 1)
@@
 		(lib_id "Alidade:SW_Push")
 		(at 248.92 82.55 0)
+		(mirror y)
 		(unit 1)
 		(body_style 1)

Commit message: i2c eeprom
Connections:
- net ROW2: now also EXSW1.2; no longer EXSW1.1
- net ROW3: now also EXSW2.2; no longer EXSW2.1
- net rROW2: now also rEXSW1.2; no longer rEXSW1.1
- net rROW3: now also rEXSW2.2; no longer rEXSW2.1
- net at D23.1 (A): now also EXSW2.1; no longer EXSW2.2
- net at D22.1 (A): now also EXSW1.1; no longer EXSW1.2
- net at rD23.1 (A): now also rEXSW2.1; no longer rEXSW2.2
- net at rD22.1 (A): now also rEXSW1.1; no longer rEXSW1.2
Changed lines of the file:
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@@
 		(lib_id "Alidade:SW_Push")
 		(at 172.72 97.79 0)
+		(mirror y)
 		(unit 1)
 		(body_style 1)
@@
 		(lib_id "Alidade:SW_Push")
 		(at 172.72 82.55 0)
+		(mirror y)
 		(unit 1)
 		(body_style 1)
@@
 		(lib_id "Alidade:SW_Push")
 		(at 248.92 97.79 0)
-		(mirror y)
 		(unit 1)
 		(body_style 1)
@@
 		(lib_id "Alidade:SW_Push")
 		(at 248.92 82.55 0)
-		(mirror y)
 		(unit 1)
 		(body_style 1)
