File: hw/mcu.kicad_sch (KiCad schematic)
At the start: 70 parts, among them J3 TC2050-IDC, U2 NRF54L15-QFAA-R, Y1 ABS07-32.768KHZ-T, Y2 ABM8G-32.000MHZ-B4Y-T

Commit message: i2c eeprom
Parts:
- added R25, R5, R6, rR25, rR5, rR6: 10k, Alidade:R_0603_1608Metric, symbol Alidade:R
- added U4, rU5: AT24C32E-STUM-T, Alidade:TSOT5_MC_MCH, symbol Alidade:AT24C32E-STUM-T
Connections:
- net PMICGPIO2 is gone; now on net PMICINT: U2.23 (P0.00)
- net rPMICGPIO2 is gone; now on net rPMICINT: rU4.23 (P0.00)
- net GND: now also U4.2 (GND)
- net PMICINT: no longer U2.27 (P0.02)
- net SCL: now also R5.2, U4.1 (SCL)
- net SDA: now also R6.2, U4.3 (SDA)
- net rDVDD: now also R25.1, R5.1, R6.1, U4.4 (VCC), rR25.1, rR5.1, rR6.1, rU5.4 (VCC)
- net rGND: now also rU5.2 (GND)
- net rPMICINT: no longer rU4.27 (P0.02)
- net rSCL: now also rR5.2, rU5.1 (SCL)
- net rSDA: now also rR6.2, rU5.3 (SDA)
- net PMICGPIO3 renamed PMICGPIO1
- net rPMICGPIO3 renamed rPMICGPIO1
- new net: R25.2, U2.27 (P0.02), U4.5 (WP)
- new net: rR25.2, rU4.27 (P0.02), rU5.5 (WP)
Other:
- note added: "Port 0 EEPROM + I2C"
- note removed: "Port 0"
- moved on the sheet: U2D, rU4D

Commit message: add ft200xd, eeprom, and esd protection
Parts:
- renumbered rU4 to rU2, rU5 to rU4
Connections:
- net DVDD: now also R25.1, R5.1, R6.1, U4.4 (VCC)
- net rDVDD: no longer R25.1, R5.1, R6.1, U4.4 (VCC)
- net rCBUS0: now reaches rU2.3 (P1.02/NFC1)
- net CBUS0: now reaches U2.3 (P1.02/NFC1)
- no-connect marks 4 -> 2
Changed lines of the file:
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@@
 	)
 	(junction
+		(at 251.46 52.07)
+		(diameter 0)
+		(color 0 0 0 0)
+	)
+	(junction
 		(at 332.74 52.07)
 		(diameter 0)
@@
 	)
 	(junction
+		(at 355.6 49.53)
+		(diameter 0)
+		(color 0 0 0 0)
+	)
+	(junction
 		(at 160.02 134.62)
 		(diameter 0)
@@
 	)
 	(junction
+		(at 351.79 52.07)
+		(diameter 0)
+		(color 0 0 0 0)
+	)
+	(junction
 		(at 41.91 83.82)
 		(diameter 0)
@@
 	)
 	(junction
+		(at 255.27 49.53)
+		(diameter 0)
+		(color 0 0 0 0)
+	)
+	(junction
 		(at 342.9 46.99)
 		(diameter 0)
@@
 	)
 	(no_connect
-		(at 359.41 110.49)
-	)
-	(no_connect
 		(at 359.41 113.03)
 	)
-	(no_connect
-		(at 281.94 109.22)
-	)
 	(wire
 		(pts
@@
 	(wire
 		(pts
-			(xy 337.82 49.53) (xy 358.14 49.53)
-		)
-		(stroke
-			(width 0)
-			(type default)
-		)
-	)
-	(wire
-		(pts
 			(xy 151.13 241.3) (xy 152.4 241.3)
 		)
@@
 	(wire
 		(pts
-			(xy 332.74 52.07) (xy 358.14 52.07)
+			(xy 332.74 52.07) (xy 351.79 52.07)
 		)
 		(stroke
@@
 	(wire
 		(pts
-			(xy 232.41 54.61) (xy 232.41 52.07)
+			(xy 251.46 54.61) (xy 251.46 52.07)
 		)
 		(stroke
@@
 	(wire
 		(pts
-			(xy 337.82 54.61) (xy 337.82 49.53)
+			(xy 355.6 54.61) (xy 355.6 49.53)
 		)
 		(stroke
@@
 	(wire
 		(pts
+			(xy 351.79 52.07) (xy 358.14 52.07)
+		)
+		(stroke
+			(width 0)
+			(type default)
+		)
+	)
+	(wire
+		(pts
 			(xy 43.18 143.51) (xy 48.26 143.51)
 		)
@@
 	(wire
 		(pts
-			(xy 332.74 54.61) (xy 332.74 52.07)
+			(xy 351.79 54.61) (xy 351.79 52.07)
 		)
 		(stroke
@@
 	(wire
 		(pts
+			(xy 337.82 49.53) (xy 358.14 49.53)
+		)
+		(stroke
+			(width 0)
+			(type default)
+		)
+	)
+	(wire
+		(pts
 			(xy 341.63 190.5) (xy 344.17 190.5)
 		)
@@
 	(wire
 		(pts
-			(xy 237.49 54.61) (xy 237.49 49.53)
+			(xy 255.27 54.61) (xy 255.27 49.53)
 		)
 		(stroke
@@
 	(hierarchical_label "SDA"
 		(shape bidirectional)
-		(at 237.49 54.61 270)
+		(at 255.27 54.61 270)
 		(effects
 			(font
@@
 		)
 	)
+	(hierarchical_label "CBUS0"
+		(shape bidirectional)
+		(at 281.94 109.22 180)
+		(effects
+			(font
+				(size 1.27 1.27)
+			)
+			(justify right)
+		)
+	)
 	(hierarchical_label "rCOL5"
 		(shape input)
@@
 	(hierarchical_label "SCL"
 		(shape output)
-		(at 232.41 54.61 270)
+		(at 251.46 54.61 270)
 		(effects
 			(font
@@
 	(hierarchical_label "rSDA"
 		(shape bidirectional)
-		(at 337.82 54.61 270)
+		(at 355.6 54.61 270)
 		(effects
 			(font
@@
 	(hierarchical_label "rSCL"
 		(shape output)
-		(at 332.74 54.61 270)
+		(at 351.79 54.61 270)
 		(effects
 			(font
@@
 		)
 	)
+	(hierarchical_label "rCBUS0"
+		(shape bidirectional)
+		(at 359.41 110.49 180)
+		(effects
+			(font
+				(size 1.27 1.27)
+			)
+			(justify right)
+		)
+	)
 	(hierarchical_label "COL4"
 		(shape input)
@@
 		(dnp no)
 		(fields_autoplaced yes)
-		(property "Reference" "rU4"
+		(property "Reference" "rU2"
 			(at 370.84 98.044 0)
 			(show_name no)
@@
 			(project "alidade"
 				(path "/4cc5d416-57f5-4147-8183-e03ae6b1198a/43e81299-cad2-4202-975b-6352d1fdfcdc"
-					(reference "rU4")
+					(reference "rU2")
 					(unit 2)
 				)
@@
 		(dnp no)
 		(fields_autoplaced yes)
-		(property "Reference" "rU4"
+		(property "Reference" "rU2"
 			(at 363.22 180.594 0)
 			(show_name no)
@@
 			(project "alidade"
 				(path "/4cc5d416-57f5-4147-8183-e03ae6b1198a/43e81299-cad2-4202-975b-6352d1fdfcdc"
-					(reference "rU4")
+					(reference "rU2")
 					(unit 3)
 				)
@@
 		(dnp no)
 		(fields_autoplaced yes)
-		(property "Reference" "rU4"
+		(property "Reference" "rU2"
 			(at 148.59 38.354 0)
 			(show_name no)
@@
 			(project "alidade"
 				(path "/4cc5d416-57f5-4147-8183-e03ae6b1198a/43e81299-cad2-4202-975b-6352d1fdfcdc"
-					(reference "rU4")
+					(reference "rU2")
 					(unit 1)
 				)
@@
 		(dnp no)
 		(fields_autoplaced yes)
-		(property "Reference" "rU4"
+		(property "Reference" "rU2"
 			(at 369.57 34.544 0)
 			(show_name no)
@@
 			(project "alidade"
 				(path "/4cc5d416-57f5-4147-8183-e03ae6b1198a/43e81299-cad2-4202-975b-6352d1fdfcdc"
-					(reference "rU4")
+					(reference "rU2")
 					(unit 4)
 				)
@@
 	)
 	(symbol
+		(lib_id "Alidade:DVDD")
+		(at 234.95 34.29 0)
+		(unit 1)
+		(body_style 1)
+		(exclude_from_sim no)
+		(in_bom yes)
+		(on_board yes)
+		(in_pos_files yes)
+		(dnp no)
+		(fields_autoplaced yes)
+		(property "Reference" "#DVDD0402"
+			(at 234.95 38.1 0)
+			(hide yes)
+			(show_name no)
+			(do_not_autoplace no)
+			(effects
+				(font
+					(size 1.27 1.27)
+				)
+			)
+		)
+		(property "Value" "DVDD"
+			(at 234.95 29.21 0)
+			(show_name no)
+			(do_not_autoplace no)
+			(effects
+				(font
+					(size 1.27 1.27)
+				)
+			)
+		)
+		(property "Footprint" ""
+			(at 234.95 34.29 0)
+			(hide yes)
+			(show_name no)
+			(do_not_autoplace no)
+			(effects
+				(font
+					(size 1.27 1.27)
+				)
+			)
+		)
+		(property "Datasheet" ""
+			(at 234.95 34.29 0)
+			(hide yes)
+			(show_name no)
+			(do_not_autoplace no)
+			(effects
+				(font
+					(size 1.27 1.27)
+				)
+			)
+		)
+		(property "Description" ""
+			(at 234.95 34.29 0)
+			(show_name no)
+			(do_not_autoplace no)
+			(effects
+				(font
+					(size 1.27 1.27)
+				)
+			)
+		)
+		(pin "1"
+		)
+		(instances
+			(project "alidade"
+				(path "/4cc5d416-57f5-4147-8183-e03ae6b1198a/43e81299-cad2-4202-975b-6352d1fdfcdc"
+					(reference "#DVDD0402")
+					(unit 1)
+				)
+			)
+		)
+	)
+	(symbol
 		(lib_id "Alidade:NRF54L15-QFAA-R")
 		(at 142.24 77.47 0)
@@
 		(dnp no)
 		(fields_autoplaced yes)
-		(property "Reference" "rU4"
+		(property "Reference" "rU2"
 			(at 153.67 72.644 0)
 			(show_name no)
@@
 			(project "alidade"
 				(path "/4cc5d416-57f5-4147-8183-e03ae6b1198a/43e81299-cad2-4202-975b-6352d1fdfcdc"
-					(reference "rU4")
+					(reference "rU2")
 					(unit 6)
 				)
@@
 	)
 	(symbol
-		(lib_id "Alidade:rDVDD")
-		(at 234.95 34.29 0)
-		(unit 1)
-		(body_style 1)
-		(exclude_from_sim no)
-		(in_bom yes)
-		(on_board yes)
-		(in_pos_files yes)
-		(dnp no)
-		(fields_autoplaced yes)
-		(property "Reference" "#rDVDD0403"
-			(at 234.95 38.1 0)
-			(hide yes)
-			(show_name no)
-			(do_not_autoplace no)
-			(effects
-				(font
-					(size 1.27 1.27)
-				)
-			)
-		)
-		(property "Value" "rDVDD"
-			(at 234.95 29.21 0)
-			(show_name no)
-			(do_not_autoplace no)
-			(effects
-				(font
-					(size 1.27 1.27)
-				)
-			)
-		)
-		(property "Footprint" ""
-			(at 234.95 34.29 0)
-			(hide yes)
-			(show_name no)
-			(do_not_autoplace no)
-			(effects
-				(font
-					(size 1.27 1.27)
-				)
-			)
-		)
-		(property "Datasheet" ""
-			(at 234.95 34.29 0)
-			(hide yes)
-			(show_name no)
-			(do_not_autoplace no)
-			(effects
-				(font
-					(size 1.27 1.27)
-				)
-			)
-		)
-		(property "Description" ""
-			(at 234.95 34.29 0)
-			(show_name no)
-			(do_not_autoplace no)
-			(effects
-				(font
-					(size 1.27 1.27)
-				)
-			)
-		)
-		(pin "1"
-		)
-		(instances
-			(project "alidade"
-				(path "/4cc5d416-57f5-4147-8183-e03ae6b1198a/43e81299-cad2-4202-975b-6352d1fdfcdc"
-					(reference "#rDVDD0403")
-					(unit 1)
-				)
-			)
-		)
-	)
-	(symbol
 		(lib_id "Alidade:NRF54L15-QFAA-R")
 		(at 200.66 132.08 0)
@@
 		(dnp no)
 		(fields_autoplaced yes)
-		(property "Reference" "rU4"
+		(property "Reference" "rU2"
 			(at 212.09 127.254 0)
 			(show_name no)
@@
 			(project "alidade"
 				(path "/4cc5d416-57f5-4147-8183-e03ae6b1198a/43e81299-cad2-4202-975b-6352d1fdfcdc"
-					(reference "rU4")
+					(reference "rU2")
 					(unit 5)
 				)
@@
 		(dnp no)
 		(fields_autoplaced yes)
-		(property "Reference" "rU5"
+		(property "Reference" "rU4"
 			(at 314.96 36.83 0)
 			(show_name no)
@@
 			(project "alidade"
 				(path "/4cc5d416-57f5-4147-8183-e03ae6b1198a/43e81299-cad2-4202-975b-6352d1fdfcdc"
-					(reference "rU5")
+					(reference "rU4")
 					(unit 1)
 				)
