File: hw/schematics/mcu.kicad_sch (KiCad schematic)
At the start: 10 parts, among them J3 TC2050-IDC, U1 ISP2454-LP-JT

Commit message: apply 0603 footprint
Parts:
- R15, R16, R17, rR15, rR16, rR17: footprint (none) -> Alidade:SMD_0603
Changed lines of the file:
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@@
 			)
 		)
-		(property "Footprint" ""
+		(property "Footprint" "Alidade:SMD_0603"
 			(at 134.62 156.21 0)
 			(effects
@@
 			)
 		)
-		(property "Footprint" ""
+		(property "Footprint" "Alidade:SMD_0603"
 			(at 147.32 156.21 0)
 			(effects
@@
 			)
 		)
-		(property "Footprint" ""
+		(property "Footprint" "Alidade:SMD_0603"
 			(at 140.97 156.21 0)
 			(effects
@@
 			)
 		)
-		(property "Footprint" ""
+		(property "Footprint" "Alidade:SMD_0603"
 			(at 62.23 157.48 0)
 			(effects
@@
 			)
 		)
-		(property "Footprint" ""
+		(property "Footprint" "Alidade:SMD_0603"
 			(at 68.58 157.48 0)
 			(effects
@@
 			)
 		)
-		(property "Footprint" ""
+		(property "Footprint" "Alidade:SMD_0603"
 			(at 55.88 157.48 0)
 			(effects

Commit message: add some LCSC part numbers
Parts:
- R15, R16, R17, rR15, rR16, rR17: footprint Alidade:SMD_0603 -> Alidade:0603; LCSC Part # (none) -> C25804
Changed lines of the file:
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@@
 			)
 		)
-		(property "JLCPCB Part #" ""
-			(at 85.09 44.45 0)
-			(effects
-				(font
-					(size 1.27 1.27)
-				)
-				(hide yes)
-			)
-		)
 		(property "LCSC Part #" "~"
 			(at 85.09 44.45 0)
@@
 			)
 		)
-		(property "Footprint" "Alidade:SMD_0603"
+		(property "Footprint" "Alidade:0603"
 			(at 134.62 156.21 0)
 			(effects
@@
 			)
 		)
-		(property "JLCPCB Part #" ""
+		(property "LCSC Part #" "C25804"
 			(at 134.62 156.21 0)
 			(effects
@@
 			)
 		)
-		(property "JLCPCB Part #" ""
-			(at 168.91 143.51 0)
-			(effects
-				(font
-					(size 1.27 1.27)
-				)
-				(hide yes)
-			)
-		)
 		(property "LCSC Part #" "~"
 			(at 168.91 143.51 0)
@@
 			)
 		)
-		(property "JLCPCB Part #" ""
-			(at 298.45 165.1 0)
-			(effects
-				(font
-					(size 1.27 1.27)
-				)
-				(hide yes)
-			)
-		)
 		(property "LCSC Part #" "~"
 			(at 298.45 165.1 0)
@@
 			)
 		)
-		(property "JLCPCB Part #" ""
-			(at 351.79 165.1 0)
-			(effects
-				(font
-					(size 1.27 1.27)
-				)
-				(hide yes)
-			)
-		)
 		(property "LCSC Part #" "~"
 			(at 351.79 165.1 0)
@@
 			)
 		)
-		(property "JLCPCB Part #" ""
-			(at 162.56 62.23 0)
-			(effects
-				(font
-					(size 1.27 1.27)
-				)
-				(hide yes)
-			)
-		)
 		(property "LCSC Part #" "~"
 			(at 162.56 62.23 0)
@@
 			)
 		)
-		(property "Footprint" "Alidade:SMD_0603"
+		(property "Footprint" "Alidade:0603"
 			(at 147.32 156.21 0)
 			(effects
@@
 			)
 		)
-		(property "JLCPCB Part #" ""
+		(property "LCSC Part #" "C25804"
 			(at 147.32 156.21 0)
 			(effects
@@
 			)
 		)
-		(property "Footprint" "Alidade:SMD_0603"
+		(property "Footprint" "Alidade:0603"
 			(at 140.97 156.21 0)
 			(effects
@@
 			)
 		)
-		(property "JLCPCB Part #" ""
+		(property "LCSC Part #" "C25804"
 			(at 140.97 156.21 0)
 			(effects
@@
 			)
 		)
-		(property "JLCPCB Part #" ""
-			(at 332.74 82.55 0)
-			(effects
-				(font
-					(size 1.27 1.27)
-				)
-				(hide yes)
-			)
-		)
 		(property "LCSC Part #" "~"
 			(at 332.74 82.55 0)
@@
 			)
 		)
-		(property "Footprint" "Alidade:SMD_0603"
+		(property "Footprint" "Alidade:0603"
 			(at 62.23 157.48 0)
 			(effects
@@
 			)
 		)
-		(property "JLCPCB Part #" ""
+		(property "LCSC Part #" "C25804"
 			(at 62.23 157.48 0)
 			(effects
@@
 			)
 		)
-		(property "JLCPCB Part #" ""
-			(at 240.03 60.96 0)
-			(effects
-				(font
-					(size 1.27 1.27)
-				)
-				(hide yes)
-			)
-		)
 		(property "LCSC Part #" "~"
 			(at 240.03 60.96 0)
@@
 			)
 		)
-		(property "JLCPCB Part #" ""
-			(at 369.57 83.82 0)
-			(effects
-				(font
-					(size 1.27 1.27)
-				)
-				(hide yes)
-			)
-		)
 		(property "LCSC Part #" "~"
 			(at 369.57 83.82 0)
@@
 			)
 		)
-		(property "JLCPCB Part #" ""
-			(at 90.17 144.78 0)
-			(effects
-				(font
-					(size 1.27 1.27)
-				)
-				(hide yes)
-			)
-		)
 		(property "LCSC Part #" "~"
 			(at 90.17 144.78 0)
@@
 			)
 		)
-		(property "JLCPCB Part #" ""
-			(at 358.14 43.18 0)
-			(effects
-				(font
-					(size 1.27 1.27)
-				)
-				(hide yes)
-			)
-		)
 		(property "LCSC Part #" "~"
 			(at 358.14 43.18 0)
@@
 			)
 		)
-		(property "JLCPCB Part #" ""
-			(at 328.93 43.18 0)
-			(effects
-				(font
-					(size 1.27 1.27)
-				)
-				(hide yes)
-			)
-		)
 		(property "LCSC Part #" "~"
 			(at 328.93 43.18 0)
@@
 			)
 		)
-		(property "JLCPCB Part #" ""
-			(at 49.53 43.18 0)
-			(effects
-				(font
-					(size 1.27 1.27)
-				)
-				(hide yes)
-			)
-		)
 		(property "LCSC Part #" "~"
 			(at 49.53 43.18 0)
@@
 			)
 		)
-		(property "Footprint" "Alidade:SMD_0603"
+		(property "Footprint" "Alidade:0603"
 			(at 68.58 157.48 0)
 			(effects
@@
 			)
 		)
-		(property "JLCPCB Part #" ""
+		(property "LCSC Part #" "C25804"
 			(at 68.58 157.48 0)
 			(effects
@@
 			)
 		)
-		(property "Footprint" "Alidade:SMD_0603"
+		(property "Footprint" "Alidade:0603"
 			(at 55.88 157.48 0)
 			(effects
@@
 			)
 		)
-		(property "JLCPCB Part #" ""
+		(property "LCSC Part #" "C25804"
 			(at 55.88 157.48 0)
 			(effects

Commit message: Remove FPGA, no longer needed
Connections:
- net CDONE: no longer names the net of U1.35 (P1.06_AIN2)
- net CRESET: no longer names the net of U1.38 (P1.05_AIN1)
- net FPGACS renamed CS
- net FPGASCK renamed SCK
- net FPGASI renamed MOSI
- net FPGASO renamed MISO
- net rCDONE: no longer names the net of rU1.35 (P1.06_AIN2)
- net rCRESET: no longer names the net of rU1.38 (P1.05_AIN1)
- net rFPGACS renamed rCS
- net rFPGASCK renamed rSCK
- net rFPGASI renamed rMISO
- net rFPGASO renamed rMOSI
Changed lines of the file:
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@@
-		)
-	)
-	(hierarchical_label "rCRESET"
-		(shape output)
-		(at 351.79 175.26 180)
-		(effects
-			(font
-				(size 1.27 1.27)
-			)
-			(justify right)
-		)
-	)
-	(hierarchical_label "CRESET"
-		(shape output)
-		(at 298.45 175.26 180)
-		(effects
-			(font
-				(size 1.27 1.27)
-			)
-			(justify right)
 		)
 	)
@@
 		)
 	)
-	(hierarchical_label "rFPGASI"
+	(hierarchical_label "rMISO"
 		(shape output)
 		(at 232.41 73.66 180)
@@
 		)
 	)
-	(hierarchical_label "CDONE"
-		(shape input)
-		(at 298.45 177.8 180)
-		(effects
-			(font
-				(size 1.27 1.27)
-			)
-			(justify right)
-		)
-	)
-	(hierarchical_label "rFPGASCK"
+	(hierarchical_label "rSCK"
 		(shape bidirectional)
 		(at 232.41 81.28 180)
@@
 		)
 	)
-	(hierarchical_label "rFPGACS"
+	(hierarchical_label "rCS"
 		(shape bidirectional)
 		(at 232.41 71.12 180)
@@
 		)
 	)
-	(hierarchical_label "FPGACS"
+	(hierarchical_label "CS"
 		(shape bidirectional)
 		(at 154.94 72.39 180)
@@
 		)
 	)
-	(hierarchical_label "rCDONE"
-		(shape input)
-		(at 351.79 177.8 180)
-		(effects
-			(font
-				(size 1.27 1.27)
-			)
-			(justify right)
-		)
-	)
-	(hierarchical_label "FPGASO"
+	(hierarchical_label "MISO"
 		(shape input)
 		(at 154.94 74.93 180)
@@
 		)
 	)
-	(hierarchical_label "FPGASI"
+	(hierarchical_label "MOSI"
 		(shape output)
 		(at 154.94 77.47 180)
@@
 		)
 	)
-	(hierarchical_label "FPGASCK"
+	(hierarchical_label "SCK"
 		(shape bidirectional)
 		(at 154.94 82.55 180)
@@
 		)
 	)
-	(hierarchical_label "rFPGASO"
+	(hierarchical_label "rMOSI"
 		(shape input)
 		(at 232.41 76.2 180)

Commit message: Update symbol, use ads122S for bridge measurement
Connections:
- net CS: no longer names the net of U1.5 (P2.10_TRACEDATA3/CSN)
- net PMICSCL renamed SCL
- net PMICSDA renamed SDA
- net rCS: no longer names the net of rU1.5 (P2.10_TRACEDATA3/CSN)
- net rPMICSCL renamed rSCL
- net rPMICSDA renamed rSDA
Other:
- note added: "Port 1 PMICSDA/SCL pulled up on PMIC sheet"
- note removed: "Port 1 PMICSDA/SCL pulled up on PMIC sheet CRESET/CDONE pulled up on FPGA sheet"
Changed lines of the file:
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@@
 		)
 	)
-	(text "Port 1\nPMICSDA/SCL pulled up on PMIC sheet\nCRESET/CDONE pulled up on FPGA sheet"
+	(text "Port 1\nPMICSDA/SCL pulled up on PMIC sheet"
 		(exclude_from_sim no)
 		(at 333.502 149.606 0)
@@
 	(wire
 		(pts
-			(xy 154.94 72.39) (xy 162.56 72.39)
-		)
-		(stroke
-			(width 0)
-			(type default)
-		)
-	)
-	(wire
-		(pts
 			(xy 82.55 69.85) (xy 85.09 69.85)
 		)
@@
 		(pts
 			(xy 158.75 158.75) (xy 168.91 158.75)
-		)
-		(stroke
-			(width 0)
-			(type default)
-		)
-	)
-	(wire
-		(pts
-			(xy 232.41 71.12) (xy 240.03 71.12)
 		)
 		(stroke
@@
 		)
 	)
-	(hierarchical_label "PMICSCL"
+	(hierarchical_label "SCL"
 		(shape output)
 		(at 298.45 170.18 180)
@@
 	)
 	(hierarchical_label "rMISO"
+		(shape input)
+		(at 232.41 73.66 180)
+		(effects
+			(font
+				(size 1.27 1.27)
+			)
+			(justify right)
+		)
+	)
+	(hierarchical_label "rSCK"
 		(shape output)
-		(at 232.41 73.66 180)
+		(at 232.41 81.28 180)
 		(effects
 			(font
@@
 		)
 	)
-	(hierarchical_label "rSCK"
-		(shape bidirectional)
-		(at 232.41 81.28 180)
-		(effects
-			(font
-				(size 1.27 1.27)
-			)
-			(justify right)
-		)
-	)
-	(hierarchical_label "rCS"
-		(shape bidirectional)
-		(at 232.41 71.12 180)
-		(effects
-			(font
-				(size 1.27 1.27)
-			)
-			(justify right)
-		)
-	)
-	(hierarchical_label "rPMICSCL"
+	(hierarchical_label "rSCL"
 		(shape output)
 		(at 351.79 170.18 180)
-		(effects
-			(font
-				(size 1.27 1.27)
-			)
-			(justify right)
-		)
-	)
-	(hierarchical_label "CS"
-		(shape bidirectional)
-		(at 154.94 72.39 180)
 		(effects
 			(font
@@
 	)
 	(hierarchical_label "SCK"
-		(shape bidirectional)
+		(shape output)
 		(at 154.94 82.55 180)
 		(effects
@@
 		)
 	)
-	(hierarchical_label "rPMICSDA"
+	(hierarchical_label "rSDA"
 		(shape bidirectional)
 		(at 351.79 167.64 180)
@@
 		)
 	)
-	(hierarchical_label "PMICSDA"
+	(hierarchical_label "SDA"
 		(shape bidirectional)
 		(at 298.45 167.64 180)
@@
 	)
 	(hierarchical_label "rMOSI"
-		(shape input)
+		(shape output)
 		(at 232.41 76.2 180)
 		(effects

Commit message: Solve erc errors
Connections:
- net rDRDY: now reaches rU1.27 (P0.01)
- net rADCCS: now reaches rU1.29 (P0.00)
- net rFAULT: now reaches rU1.32 (P0.02)
- net DRDY: now reaches U1.27 (P0.01)
- net ADCCS: now reaches U1.29 (P0.00)
- net FAULT: now reaches U1.32 (P0.02)
Changed lines of the file:
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@@
 	)
 	(no_connect
-		(at 358.14 55.88)
-	)
-	(no_connect
 		(at 332.74 133.35)
 	)
@@
 	)
 	(no_connect
+		(at 298.45 177.8)
+	)
+	(no_connect
 		(at 351.79 198.12)
 	)
@@
 	)
 	(no_connect
+		(at 358.14 53.34)
+	)
+	(no_connect
+		(at 240.03 71.12)
+	)
+	(no_connect
 		(at 351.79 185.42)
 	)
@@
 	)
 	(no_connect
-		(at 369.57 127)
+		(at 351.79 177.8)
 	)
 	(no_connect
-		(at 328.93 48.26)
+		(at 369.57 127)
 	)
 	(no_connect
@@
 	)
 	(no_connect
-		(at 358.14 48.26)
-	)
-	(no_connect
 		(at 369.57 114.3)
 	)
@@
 	)
 	(no_connect
-		(at 358.14 53.34)
-	)
-	(no_connect
 		(at 369.57 109.22)
 	)
 	(no_connect
-		(at 358.14 45.72)
-	)
-	(no_connect
 		(at 369.57 124.46)
 	)
@@
 	)
 	(no_connect
+		(at 298.45 175.26)
+	)
+	(no_connect
 		(at 298.45 190.5)
 	)
@@
 	)
 	(no_connect
-		(at 369.57 119.38)
+		(at 162.56 72.39)
 	)
 	(no_connect
-		(at 328.93 50.8)
-	)
-	(no_connect
-		(at 358.14 50.8)
+		(at 358.14 55.88)
 	)
 	(no_connect
-		(at 328.93 45.72)
+		(at 369.57 119.38)
 	)
 	(no_connect
@@
 		(at 369.57 96.52)
 	)
+	(no_connect
+		(at 351.79 175.26)
+	)
 	(wire
 		(pts
@@
 		)
 	)
+	(hierarchical_label "rFAULT"
+		(shape input)
+		(at 358.14 50.8 180)
+		(effects
+			(font
+				(size 1.27 1.27)
+			)
+			(justify right)
+		)
+	)
+	(hierarchical_label "FAULT"
+		(shape input)
+		(at 328.93 50.8 180)
+		(effects
+			(font
+				(size 1.27 1.27)
+			)
+			(justify right)
+		)
+	)
+	(hierarchical_label "rADCCS"
+		(shape output)
+		(at 358.14 45.72 180)
+		(effects
+			(font
+				(size 1.27 1.27)
+			)
+			(justify right)
+		)
+	)
+	(hierarchical_label "DRDY"
+		(shape input)
+		(at 328.93 48.26 180)
+		(effects
+			(font
+				(size 1.27 1.27)
+			)
+			(justify right)
+		)
+	)
 	(hierarchical_label "rSCK"
 		(shape output)
@@
 		)
 	)
+	(hierarchical_label "rDRDY"
+		(shape input)
+		(at 358.14 48.26 180)
+		(effects
+			(font
+				(size 1.27 1.27)
+			)
+			(justify right)
+		)
+	)
 	(hierarchical_label "MOSI"
 		(shape output)
@@
 		)
 	)
+	(hierarchical_label "ADCCS"
+		(shape output)
+		(at 328.93 45.72 180)
+		(effects
+			(font
+				(size 1.27 1.27)
+			)
+			(justify right)
+		)
+	)
 	(hierarchical_label "rSDA"
 		(shape bidirectional)
@@
 			)
 		)
-		(property "Description" ""
+		(property "Description" "TAG Connect Receptacle"
 			(at 168.91 143.51 0)
 			(effects
@@
 			)
 		)
-		(property "Description" ""
+		(property "Description" "TAG Connect Receptacle"
 			(at 90.17 144.78 0)
 			(effects
