File: hw/schematics/mcu.kicad_sch (KiCad schematic)
At the start: 70 parts, among them J3 TC2050-IDC, U2 NRF54L15-QFAA-R, Y1 32.768K, Y2 32M

Commit message: Add extra pmic gpios
Connections:
- net PMICGPIO2: now reaches U2.23 (P0.00)
- net PMICGPIO3: now reaches U2.24 (P0.01)
- net rPMICGPIO2: now reaches rU4.23 (P0.00)
- net rPMICGPIO3: now reaches rU4.24 (P0.01)
- no-connect marks 8 -> 4
Changed lines of the file:
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@@
 	)
 	(no_connect
-		(at 276.86 41.91)
-	)
-	(no_connect
 		(at 281.94 111.76)
 	)
@@
 	)
 	(no_connect
-		(at 332.74 44.45)
-	)
-	(no_connect
 		(at 359.41 113.03)
 	)
 	(no_connect
-		(at 276.86 44.45)
-	)
-	(no_connect
-		(at 332.74 41.91)
-	)
-	(no_connect
 		(at 281.94 109.22)
 	)
@@
 		)
 	)
+	(hierarchical_label "rPMICGPIO3"
+		(shape bidirectional)
+		(at 332.74 44.45 180)
+		(effects
+			(font
+				(size 1.27 1.27)
+			)
+			(justify right)
+		)
+	)
 	(hierarchical_label "rCOL5"
 		(shape input)
@@
 		)
 	)
+	(hierarchical_label "PMICGPIO3"
+		(shape bidirectional)
+		(at 276.86 44.45 180)
+		(effects
+			(font
+				(size 1.27 1.27)
+			)
+			(justify right)
+		)
+	)
+	(hierarchical_label "rPMICGPIO2"
+		(shape bidirectional)
+		(at 332.74 41.91 180)
+		(effects
+			(font
+				(size 1.27 1.27)
+			)
+			(justify right)
+		)
+	)
 	(hierarchical_label "rROW4"
 		(shape output)
@@
 		(effects
 			(font
+				(size 1.27 1.27)
+			)
+			(justify right)
+		)
+	)
+	(hierarchical_label "PMICGPIO2"
+		(shape bidirectional)
+		(at 276.86 41.91 180)
+		(effects
+			(font

Commit message: Add a bunch of models and footprints
Parts:
- ANT1: footprint (none) -> Alidade:Texas_SWRA117D_2.4GHz_Left
- C12, C13, C14, C15, C16, C17, C18, C19, C20, C21, C22, C23, rC12, rC13, rC14, rC15, rC16, rC17, rC18, rC19, rC20, rC21, rC22, rC23: footprint (none) -> Alidade:C_0603_1608Metric
- FB1, L3, L4, L5, L6, rFB1, rL3, rL4, rL5, rL6: footprint (none) -> Alidade:L_0603_1608Metric
- R17, R18, R19, R20, R21, R22, R23, R24, rR17, rR18, rR19, rR20, rR21, rR22, rR23, rR24: footprint Alidade:0603 -> Alidade:R_0603_1608Metric
- TP1, TP2, TP3, TP4, TP5, rTP1, rTP2, rTP3, rTP4, rTP5: footprint (none) -> Alidade:TestPoint_Pad_1.0x1.0mm
- rANT1: footprint (none) -> Alidade:Texas_SWRA117D_2.4GHz_Right
Changed lines of the file:
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@@
 			)
 		)
-		(property "Footprint" "Alidade:0603"
+		(property "Footprint" "Alidade:R_0603_1608Metric"
 			(at 346.71 198.12 0)
 			(effects
@@
 			)
 		)
-		(property "Footprint" ""
+		(property "Footprint" "Alidade:C_0603_1608Metric"
 			(at 55.88 139.7 0)
 			(effects
@@
 			)
 		)
-		(property "Footprint" ""
+		(property "Footprint" "Alidade:L_0603_1608Metric"
 			(at 118.11 85.09 0)
 			(effects
@@
 			)
 		)
-		(property "Footprint" ""
+		(property "Footprint" "Alidade:L_0603_1608Metric"
 			(at 45.72 81.28 0)
 			(effects
@@
 			)
 		)
-		(property "Footprint" ""
+		(property "Footprint" "Alidade:L_0603_1608Metric"
 			(at 52.07 135.89 0)
 			(effects
@@
 			)
 		)
-		(property "Footprint" ""
+		(property "Footprint" "Alidade:TestPoint_Pad_1.0x1.0mm"
 			(at 255.27 208.28 0)
 			(effects
@@
 			)
 		)
-		(property "Footprint" ""
+		(property "Footprint" "Alidade:C_0603_1608Metric"
 			(at 66.04 93.98 0)
 			(effects
@@
 			)
 		)
-		(property "Footprint" "Alidade:0603"
+		(property "Footprint" "Alidade:R_0603_1608Metric"
 			(at 68.58 234.95 0)
 			(effects
@@
 			)
 		)
-		(property "Footprint" ""
+		(property "Footprint" "Alidade:C_0603_1608Metric"
 			(at 46.99 53.34 0)
 			(effects
@@
 			)
 		)
-		(property "Footprint" "Alidade:0603"
+		(property "Footprint" "Alidade:R_0603_1608Metric"
 			(at 118.11 231.14 0)
 			(effects
@@
 			)
 		)
-		(property "Footprint" ""
+		(property "Footprint" "Alidade:TestPoint_Pad_1.0x1.0mm"
 			(at 344.17 200.66 0)
 			(effects
@@
 			)
 		)
-		(property "Footprint" ""
+		(property "Footprint" "Alidade:L_0603_1608Metric"
 			(at 59.69 135.89 0)
 			(effects
@@
 			)
 		)
-		(property "Footprint" ""
+		(property "Footprint" "Alidade:C_0603_1608Metric"
 			(at 160.02 138.43 0)
 			(effects
@@
 			)
 		)
-		(property "Footprint" "Alidade:0603"
+		(property "Footprint" "Alidade:R_0603_1608Metric"
 			(at 147.32 228.6 0)
 			(effects
@@
 			)
 		)
-		(property "Footprint" ""
+		(property "Footprint" "Alidade:C_0603_1608Metric"
 			(at 175.26 138.43 0)
 			(effects
@@
 			)
 		)
-		(property "Footprint" ""
+		(property "Footprint" "Alidade:C_0603_1608Metric"
 			(at 53.34 53.34 0)
 			(effects
@@
 			)
 		)
-		(property "Footprint" "Alidade:0603"
+		(property "Footprint" "Alidade:R_0603_1608Metric"
 			(at 257.81 198.12 0)
 			(effects
@@
 			)
 		)
-		(property "Footprint" "Alidade:0603"
+		(property "Footprint" "Alidade:R_0603_1608Metric"
 			(at 147.32 233.68 0)
 			(effects
@@
 			)
 		)
-		(property "Footprint" ""
+		(property "Footprint" "Alidade:C_0603_1608Metric"
 			(at 40.64 53.34 0)
 			(effects
@@
 			)
 		)
-		(property "Footprint" ""
+		(property "Footprint" "Alidade:TestPoint_Pad_1.0x1.0mm"
 			(at 255.27 198.12 0)
 			(effects
@@
 			)
 		)
-		(property "Footprint" ""
+		(property "Footprint" "Alidade:C_0603_1608Metric"
 			(at 120.65 53.34 0)
 			(effects
@@
 			)
 		)
-		(property "Footprint" "Alidade:0603"
+		(property "Footprint" "Alidade:R_0603_1608Metric"
 			(at 147.32 223.52 0)
 			(effects
@@
 			)
 		)
-		(property "Footprint" ""
+		(property "Footprint" "Alidade:C_0603_1608Metric"
 			(at 48.26 139.7 0)
 			(effects
@@
 			)
 		)
-		(property "Footprint" ""
+		(property "Footprint" "Alidade:C_0603_1608Metric"
 			(at 63.5 139.7 0)
 			(effects
@@
 			)
 		)
-		(property "Footprint" ""
+		(property "Footprint" "Alidade:C_0603_1608Metric"
 			(at 167.64 138.43 0)
 			(effects
@@
 			)
 		)
-		(property "Footprint" "Alidade:0603"
+		(property "Footprint" "Alidade:R_0603_1608Metric"
 			(at 68.58 224.79 0)
 			(effects
@@
 			)
 		)
-		(property "Footprint" ""
+		(property "Footprint" "Alidade:L_0603_1608Metric"
 			(at 179.07 134.62 0)
 			(effects
@@
 			)
 		)
-		(property "Footprint" ""
+		(property "Footprint" "Alidade:C_0603_1608Metric"
 			(at 53.34 93.98 0)
 			(effects
@@
 			)
 		)
-		(property "Footprint" ""
+		(property "Footprint" "Alidade:L_0603_1608Metric"
 			(at 45.72 86.36 0)
 			(effects
@@
 			)
 		)
-		(property "Footprint" ""
+		(property "Footprint" "Alidade:L_0603_1608Metric"
 			(at 118.11 80.01 0)
 			(effects
@@
 			)
 		)
-		(property "Footprint" "Alidade:0603"
+		(property "Footprint" "Alidade:R_0603_1608Metric"
 			(at 130.81 231.14 0)
 			(effects
@@
 			)
 		)
-		(property "Footprint" ""
+		(property "Footprint" "Alidade:TestPoint_Pad_1.0x1.0mm"
 			(at 344.17 208.28 0)
 			(effects
@@
 			)
 		)
-		(property "Footprint" ""
+		(property "Footprint" "Alidade:Texas_SWRA117D_2.4GHz_Left"
 			(at 39.37 130.81 0)
 			(effects
@@
 			)
 		)
-		(property "Footprint" ""
+		(property "Footprint" "Alidade:Texas_SWRA117D_2.4GHz_Right"
 			(at 151.13 129.54 0)
 			(effects
@@
 			)
 		)
-		(property "Footprint" ""
+		(property "Footprint" "Alidade:C_0603_1608Metric"
 			(at 36.83 93.98 0)
 			(effects
@@
 			)
 		)
-		(property "Footprint" "Alidade:0603"
+		(property "Footprint" "Alidade:R_0603_1608Metric"
 			(at 124.46 231.14 0)
 			(effects
@@
 			)
 		)
-		(property "Footprint" "Alidade:0603"
+		(property "Footprint" "Alidade:R_0603_1608Metric"
 			(at 346.71 190.5 0)
 			(effects
@@
 			)
 		)
-		(property "Footprint" ""
+		(property "Footprint" "Alidade:C_0603_1608Metric"
 			(at 132.08 92.71 0)
 			(effects
@@
 			)
 		)
-		(property "Footprint" ""
+		(property "Footprint" "Alidade:TestPoint_Pad_1.0x1.0mm"
 			(at 255.27 205.74 0)
 			(effects
@@
 			)
 		)
-		(property "Footprint" ""
+		(property "Footprint" "Alidade:TestPoint_Pad_1.0x1.0mm"
 			(at 344.17 205.74 0)
 			(effects
@@
 			)
 		)
-		(property "Footprint" "Alidade:0603"
+		(property "Footprint" "Alidade:R_0603_1608Metric"
 			(at 257.81 190.5 0)
 			(effects
@@
 			)
 		)
-		(property "Footprint" "Alidade:0603"
+		(property "Footprint" "Alidade:R_0603_1608Metric"
 			(at 45.72 232.41 0)
 			(effects
@@
 			)
 		)
-		(property "Footprint" ""
+		(property "Footprint" "Alidade:C_0603_1608Metric"
 			(at 101.6 53.34 0)
 			(effects
@@
 			)
 		)
-		(property "Footprint" ""
+		(property "Footprint" "Alidade:C_0603_1608Metric"
 			(at 59.69 93.98 0)
 			(effects
@@
 			)
 		)
-		(property "Footprint" ""
+		(property "Footprint" "Alidade:C_0603_1608Metric"
 			(at 138.43 92.71 0)
 			(effects
@@
 			)
 		)
-		(property "Footprint" ""
+		(property "Footprint" "Alidade:L_0603_1608Metric"
 			(at 171.45 134.62 0)
 			(effects
@@
 			)
 		)
-		(property "Footprint" ""
+		(property "Footprint" "Alidade:C_0603_1608Metric"
 			(at 125.73 92.71 0)
 			(effects
@@
 			)
 		)
-		(property "Footprint" ""
+		(property "Footprint" "Alidade:L_0603_1608Metric"
 			(at 67.31 135.89 0)
 			(effects
@@
 			)
 		)
-		(property "Footprint" ""
+		(property "Footprint" "Alidade:L_0603_1608Metric"
 			(at 163.83 134.62 0)
 			(effects
@@
 			)
 		)
-		(property "Footprint" ""
+		(property "Footprint" "Alidade:C_0603_1608Metric"
 			(at 107.95 53.34 0)
 			(effects
@@
 			)
 		)
-		(property "Footprint" ""
+		(property "Footprint" "Alidade:TestPoint_Pad_1.0x1.0mm"
 			(at 255.27 203.2 0)
 			(effects
@@
 			)
 		)
-		(property "Footprint" ""
+		(property "Footprint" "Alidade:TestPoint_Pad_1.0x1.0mm"
 			(at 344.17 203.2 0)
 			(effects
@@
 			)
 		)
-		(property "Footprint" ""
+		(property "Footprint" "Alidade:C_0603_1608Metric"
 			(at 109.22 92.71 0)
 			(effects
@@
 			)
 		)
-		(property "Footprint" ""
+		(property "Footprint" "Alidade:C_0603_1608Metric"
 			(at 34.29 53.34 0)
 			(effects
@@
 			)
 		)
-		(property "Footprint" ""
+		(property "Footprint" "Alidade:TestPoint_Pad_1.0x1.0mm"
 			(at 255.27 200.66 0)
 			(effects
@@
 			)
 		)
-		(property "Footprint" "Alidade:0603"
+		(property "Footprint" "Alidade:R_0603_1608Metric"
 			(at 68.58 229.87 0)
 			(effects
@@
 			)
 		)
-		(property "Footprint" ""
+		(property "Footprint" "Alidade:C_0603_1608Metric"
 			(at 127 53.34 0)
 			(effects
@@
 			)
 		)
-		(property "Footprint" ""
+		(property "Footprint" "Alidade:C_0603_1608Metric"
 			(at 114.3 53.34 0)
 			(effects
@@
 			)
 		)
-		(property "Footprint" ""
+		(property "Footprint" "Alidade:TestPoint_Pad_1.0x1.0mm"
 			(at 344.17 198.12 0)
 			(effects
@@
 			)
 		)
-		(property "Footprint" ""
+		(property "Footprint" "Alidade:C_0603_1608Metric"
 			(at 59.69 53.34 0)
 			(effects
@@
 			)
 		)
-		(property "Footprint" "Alidade:0603"
+		(property "Footprint" "Alidade:R_0603_1608Metric"
 			(at 52.07 232.41 0)
 			(effects
@@
 			)
 		)
-		(property "Footprint" "Alidade:0603"
+		(property "Footprint" "Alidade:R_0603_1608Metric"
 			(at 39.37 232.41 0)
 			(effects

Commit message: Various footprint updates
Parts:
- removed Y1, rY1: 32.768K, symbol Alidade:Crystal_GND24
- added Y1, rY1: ABS07-32.768KHZ-T, symbol Alidade:Crystal
- R21, R22, R23, rR21, rR22, rR23: LCSC Part # C25804 -> (none)
- U2, rU4: footprint Alidade:QFN48_6X6_NOR -> Alidade:QFN48_6X6; LCSC Part # (none) -> C42458750
- Y2, rY2: value 32M -> ABM8G-32.000MHZ-B4Y-T; LCSC Part # (none) -> C5187559
Connections:
- net at rU4.1 (P1.00/XL1): now also rY1.2
- net at rU4.2 (P1.01/XL2): now also rY1.1
- net at U2.1 (P1.00/XL1): now also Y1.2
- net at U2.2 (P1.01/XL2): now also Y1.1

Commit message: All footprints
Parts:
- ANT1, rANT1: value ~ -> SWRA117D
- Y1, rY1: footprint (none) -> Alidade:XTAL_ABS07-32.768KHZ-1-T
- Y2, rY2: footprint (none) -> Alidade:XTAL_ABM8G-32.000MHZ-B4Y-T
Changed lines of the file:
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@@
 			)
 		)
-		(property "Footprint" ""
+		(property "Footprint" "Alidade:XTAL_ABM8G-32.000MHZ-B4Y-T"
 			(at 195.58 147.32 0)
 			(effects
@@
 			)
 		)
-		(property "Footprint" ""
+		(property "Footprint" "Alidade:XTAL_ABM8G-32.000MHZ-B4Y-T"
 			(at 83.82 148.59 0)
 			(effects
@@
 			)
 		)
-		(property "Footprint" ""
+		(property "Footprint" "Alidade:XTAL_ABS07-32.768KHZ-1-T"
 			(at 347.98 105.41 0)
 			(effects
@@
 			)
 		)
-		(property "Value" "~"
+		(property "Value" "SWRA117D"
 			(at 27.94 142.2399 0)
 			(effects
@@
 			)
 		)
-		(property "Value" "~"
+		(property "Value" "SWRA117D"
 			(at 139.7 140.9699 0)
 			(effects
@@
 			)
 		)
-		(property "Footprint" ""
+		(property "Footprint" "Alidade:XTAL_ABS07-32.768KHZ-1-T"
 			(at 270.51 104.14 0)
 			(effects

Commit message: LCSC part numbers
Parts:
- C12, C13, C14, C15, rC12, rC13, rC14, rC15: LCSC Part # (none) -> C14663
- C16, rC16: LCSC Part # (none) -> C96446
- C17, C18, rC17, rC18: LCSC Part # (none) -> C23630
- C19, rC19: LCSC Part # (none) -> C57112
- C20, rC20: LCSC Part # (none) -> C1604
- C21, rC21: LCSC Part # (none) -> C53514
- C22, rC22: LCSC Part # (none) -> C1650
- C23, rC23: LCSC Part # (none) -> C1639
- FB1, rFB1: LCSC Part # (none) -> C1002
- L3, rL3: LCSC Part # (none) -> C1034
- L4, L5, rL4, rL5: LCSC Part # (none) -> C370237
- L6, rL6: LCSC Part # (none) -> C13817
- R17, R18, R19, R20, R24, rR17, rR18, rR19, rR20, rR24: LCSC Part # (none) -> C21189
- R21, R22, R23, rR21, rR22, rR23: LCSC Part # (none) -> C25804

Commit message: mcu r
Connections:
- net GND: no longer rANT1.2 (GND), rC21.2, rC22.2, rC23.2, rU4.32 (VSS_PA), rY2.2, rY2.4
- net rGND: now also rANT1.2 (GND), rC21.2, rC22.2, rC23.2, rU4.32 (VSS_PA), rY2.2, rY2.4
Changed lines of the file:
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@@
 	)
 	(symbol
-		(lib_id "Alidade:GND")
-		(at 163.83 143.51 0)
+		(lib_id "Alidade:rGND")
+		(at 186.69 138.43 0)
 		(unit 1)
 		(exclude_from_sim no)
@@
 		(dnp no)
 		(fields_autoplaced yes)
-		(property "Reference" "#GND0403"
-			(at 163.83 149.86 0)
+		(property "Reference" "#rGND08"
+			(at 186.69 144.78 0)
 			(effects
 				(font
@@
 			)
 		)
-		(property "Value" "GND"
-			(at 163.83 148.59 0)
+		(property "Value" "rGND"
+			(at 186.69 143.51 0)
 			(effects
 				(font
@@
 		)
 		(property "Footprint" ""
-			(at 163.83 143.51 0)
+			(at 186.69 138.43 0)
 			(effects
 				(font
@@
 		)
 		(property "Datasheet" ""
-			(at 163.83 143.51 0)
+			(at 186.69 138.43 0)
 			(effects
 				(font
@@
 		)
 		(property "Description" ""
-			(at 163.83 143.51 0)
+			(at 186.69 138.43 0)
 			(effects
 				(font
@@
 			(project "alidade"
 				(path "/4cc5d416-57f5-4147-8183-e03ae6b1198a/43e81299-cad2-4202-975b-6352d1fdfcdc"
-					(reference "#GND0403")
+					(reference "#rGND08")
 					(unit 1)
 				)
@@
 	)
 	(symbol
-		(lib_id "Alidade:GND")
-		(at 205.74 152.4 0)
-		(unit 1)
-		(exclude_from_sim no)
-		(in_bom yes)
-		(on_board yes)
-		(dnp no)
-		(fields_autoplaced yes)
-		(property "Reference" "#GND0405"
-			(at 205.74 158.75 0)
-			(effects
-				(font
-					(size 1.27 1.27)
-				)
-				(hide yes)
-			)
-		)
-		(property "Value" "GND"
-			(at 205.74 157.48 0)
-			(effects
-				(font
-					(size 1.27 1.27)
-				)
-			)
-		)
-		(property "Footprint" ""
-			(at 205.74 152.4 0)
-			(effects
-				(font
-					(size 1.27 1.27)
-				)
-				(hide yes)
-			)
-		)
-		(property "Datasheet" ""
-			(at 205.74 152.4 0)
-			(effects
-				(font
-					(size 1.27 1.27)
-				)
-				(hide yes)
-			)
-		)
-		(property "Description" ""
-			(at 205.74 152.4 0)
-			(effects
-				(font
-					(size 1.27 1.27)
-				)
-			)
-		)
-		(pin "1"
-		)
-		(instances
-			(project "alidade"
-				(path "/4cc5d416-57f5-4147-8183-e03ae6b1198a/43e81299-cad2-4202-975b-6352d1fdfcdc"
-					(reference "#GND0405")
-					(unit 1)
-				)
-			)
-		)
-	)
-	(symbol
 		(lib_id "Alidade:rDVDD")
 		(at 118.11 219.71 0)
@@
 	)
 	(symbol
-		(lib_id "Alidade:GND")
-		(at 186.69 138.43 0)
-		(unit 1)
-		(exclude_from_sim no)
-		(in_bom yes)
-		(on_board yes)
-		(dnp no)
-		(fields_autoplaced yes)
-		(property "Reference" "#GND0404"
-			(at 186.69 144.78 0)
-			(effects
-				(font
-					(size 1.27 1.27)
-				)
-				(hide yes)
-			)
-		)
-		(property "Value" "GND"
-			(at 186.69 143.51 0)
-			(effects
-				(font
-					(size 1.27 1.27)
-				)
-			)
-		)
-		(property "Footprint" ""
-			(at 186.69 138.43 0)
-			(effects
-				(font
-					(size 1.27 1.27)
-				)
-				(hide yes)
-			)
-		)
-		(property "Datasheet" ""
-			(at 186.69 138.43 0)
-			(effects
-				(font
-					(size 1.27 1.27)
-				)
-				(hide yes)
-			)
-		)
-		(property "Description" ""
-			(at 186.69 138.43 0)
-			(effects
-				(font
-					(size 1.27 1.27)
-				)
-			)
-		)
-		(pin "1"
-		)
-		(instances
-			(project "alidade"
-				(path "/4cc5d416-57f5-4147-8183-e03ae6b1198a/43e81299-cad2-4202-975b-6352d1fdfcdc"
-					(reference "#GND0404")
-					(unit 1)
-				)
-			)
-		)
-	)
-	(symbol
 		(lib_id "Alidade:SWRA117D")
 		(at 151.13 129.54 0)
@@
 	)
 	(symbol
+		(lib_id "Alidade:rGND")
+		(at 163.83 143.51 0)
+		(unit 1)
+		(exclude_from_sim no)
+		(in_bom yes)
+		(on_board yes)
+		(dnp no)
+		(fields_autoplaced yes)
+		(property "Reference" "#rGND06"
+			(at 163.83 149.86 0)
+			(effects
+				(font
+					(size 1.27 1.27)
+				)
+				(hide yes)
+			)
+		)
+		(property "Value" "rGND"
+			(at 163.83 148.59 0)
+			(effects
+				(font
+					(size 1.27 1.27)
+				)
+			)
+		)
+		(property "Footprint" ""
+			(at 163.83 143.51 0)
+			(effects
+				(font
+					(size 1.27 1.27)
+				)
+				(hide yes)
+			)
+		)
+		(property "Datasheet" ""
+			(at 163.83 143.51 0)
+			(effects
+				(font
+					(size 1.27 1.27)
+				)
+				(hide yes)
+			)
+		)
+		(property "Description" ""
+			(at 163.83 143.51 0)
+			(effects
+				(font
+					(size 1.27 1.27)
+				)
+			)
+		)
+		(pin "1"
+		)
+		(instances
+			(project "alidade"
+				(path "/4cc5d416-57f5-4147-8183-e03ae6b1198a/43e81299-cad2-4202-975b-6352d1fdfcdc"
+					(reference "#rGND06")
+					(unit 1)
+				)
+			)
+		)
+	)
+	(symbol
 		(lib_id "Alidade:L")
 		(at 163.83 134.62 90)
@@
 					(unit 1)
 				)
+			)
+		)
+	)
+	(symbol
+		(lib_id "Alidade:rGND")
+		(at 205.74 152.4 0)
+		(unit 1)
+		(exclude_from_sim no)
+		(in_bom yes)
+		(on_board yes)
+		(dnp no)
+		(fields_autoplaced yes)
+		(property "Reference" "#rGND010"
+			(at 205.74 158.75 0)
+			(effects
+				(font
+					(size 1.27 1.27)
+				)
+				(hide yes)
+			)
+		)
+		(property "Value" "rGND"
+			(at 205.74 157.48 0)
+			(effects
+				(font
+					(size 1.27 1.27)
+				)
+			)
+		)
+		(property "Footprint" ""
+			(at 205.74 152.4 0)
+			(effects
+				(font
+					(size 1.27 1.27)
+				)
+				(hide yes)
+			)
+		)
+		(property "Datasheet" ""
+			(at 205.74 152.4 0)
+			(effects
+				(font
+					(size 1.27 1.27)
+				)
+				(hide yes)
+			)
+		)
+		(property "Description" ""
+			(at 205.74 152.4 0)
+			(effects
+				(font
+					(size 1.27 1.27)
+				)
+			)
+		)
+		(pin "1"
+		)
+		(instances
+			(project "alidade"
+				(path "/4cc5d416-57f5-4147-8183-e03ae6b1198a/43e81299-cad2-4202-975b-6352d1fdfcdc"
+					(reference "#rGND010")
+					(unit 1)
+				)
