File: hw/schematics/pmic.kicad_sch (KiCad schematic)
At the start: 40 parts, among them J1 TYPE-C-31-M-13C, J2 JST_S2B-PH-SM4-TB, U1 NPM1300-QEAA-R

Commit message: pmic left
Parts:
- removed R1, rR1: 10k, Alidade:R_0603_1608Metric, symbol Alidade:R
Connections:
- net GND: now also U1.18 (NTC)
- net rGND: now also rU1.18 (NTC)
Changed lines of the file:
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@@
 	(wire
 		(pts
-			(xy 353.06 69.85) (xy 354.33 69.85)
+			(xy 353.06 69.85) (xy 359.41 69.85)
 		)
 		(stroke
@@
 	(wire
 		(pts
-			(xy 281.94 68.58) (xy 283.21 68.58)
+			(xy 281.94 68.58) (xy 288.29 68.58)
 		)
 		(stroke
@@
 	)
 	(symbol
-		(lib_id "Alidade:R")
-		(at 356.87 69.85 90)
-		(unit 1)
-		(exclude_from_sim no)
-		(in_bom yes)
-		(on_board yes)
-		(dnp no)
-		(property "Reference" "rR1"
-			(at 356.87 73.66 90)
-			(effects
-				(font
-					(size 1.27 1.27)
-				)
-			)
-		)
-		(property "Value" "10k"
-			(at 356.87 71.628 90)
-			(do_not_autoplace yes)
-			(effects
-				(font
-					(size 1.27 1.27)
-				)
-			)
-		)
-		(property "Footprint" "Alidade:R_0603_1608Metric"
-			(at 356.87 69.85 0)
-			(effects
-				(font
-					(size 1.27 1.27)
-				)
-				(hide yes)
-			)
-		)
-		(property "Datasheet" "~"
-			(at 356.87 69.85 0)
-			(effects
-				(font
-					(size 1.27 1.27)
-				)
-				(hide yes)
-			)
-		)
-		(property "Description" ""
-			(at 356.87 69.85 0)
-			(effects
-				(font
-					(size 1.27 1.27)
-				)
-				(hide yes)
-			)
-		)
-		(property "LCSC Part #" "C25804"
-			(at 356.87 69.85 90)
-			(effects
-				(font
-					(size 1.27 1.27)
-				)
-				(hide yes)
-			)
-		)
-		(pin "1"
-		)
-		(pin "2"
-		)
-		(instances
-			(project "alidade"
-				(path "/4cc5d416-57f5-4147-8183-e03ae6b1198a/29a12dcc-0491-44a2-8290-cbef7c573a8c"
-					(reference "rR1")
-					(unit 1)
-				)
-			)
-		)
-	)
-	(symbol
 		(lib_id "Alidade:NPM1300-QEAA-R")
 		(at 53.34 229.87 0)
@@
 					(unit 1)
 				)
-			)
-		)
-	)
-	(symbol
-		(lib_id "Alidade:R")
-		(at 285.75 68.58 90)
-		(unit 1)
-		(exclude_from_sim no)
-		(in_bom yes)
-		(on_board yes)
-		(dnp no)
-		(property "Reference" "R1"
-			(at 285.75 72.39 90)
-			(effects
-				(font
-					(size 1.27 1.27)
-				)
-			)
-		)
-		(property "Value" "10k"
-			(at 285.75 70.358 90)
-			(do_not_autoplace yes)
-			(effects
-				(font
-					(size 1.27 1.27)
-				)
-			)
-		)
-		(property "Footprint" "Alidade:R_0603_1608Metric"
-			(at 285.75 68.58 0)
-			(effects
-				(font
-					(size 1.27 1.27)
-				)
-				(hide yes)
-			)
-		)
-		(property "Datasheet" "~"
-			(at 285.75 68.58 0)
-			(effects
-				(font
-					(size 1.27 1.27)
-				)
-				(hide yes)
-			)
-		)
-		(property "Description" ""
-			(at 285.75 68.58 0)
-			(effects
-				(font
-					(size 1.27 1.27)
-				)
-				(hide yes)
-			)
-		)
-		(property "LCSC Part #" "C25804"
-			(at 285.75 68.58 90)
-			(effects
-				(font
-					(size 1.27 1.27)
-				)
-				(hide yes)
-			)
-		)
-		(pin "1"
-		)
-		(pin "2"
-		)
-		(instances
-			(project "alidade"
-				(path "/4cc5d416-57f5-4147-8183-e03ae6b1198a/29a12dcc-0491-44a2-8290-cbef7c573a8c"
-					(reference "R1")
-					(unit 1)
-				)

Commit message: trackpoint l
Connections:
- net rVBUS: no longer names the net of rC1.1, rJ1.A4 (VBUS), rJ1.A9 (VBUS), rJ1.B4 (VBUS), rJ1.B9 (VBUS), rU1.21 (VBUS)
Changed lines of the file:
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@@
-		)
-	)
-	(label "rVBUS"
-		(at 184.15 48.26 0)
-		(effects
-			(font
-				(size 1.27 1.27)
-			)
-			(justify left bottom)
 		)
 	)
